Commit message: gazebo model

File: erica_description/urdf/erica_robot.xacro (robot description, xacro)
@@ -45,5 +45,5 @@
   <!-- left_arm -->
   <!-- left_arm_pitch -->
- <joint name="l_arm_shoulder_pitch" type="revolute">
+ <joint name="l_arm_sh_p" type="revolute">
     <parent link="body_main"/>
     <child link="l_arm_shoulder_pitch_link"/>
@@ -53,10 +53,10 @@
     <dynamics damping = "0.7"/>
   </joint>
-  <transmission name="l_arm_shoulder_pitch_tran">
-     <type>transmission_interface/SimpleTransmission</type>
-     <joint name="l_arm_shoulder_pitch">
-       <hardwareInterface>EffortJointInterface</hardwareInterface>
-     </joint>
-     <actuator name="l_arm_shoulder_pitch_motor">
+  <transmission name="l_arm_sh_p_tran">
+     <type>transmission_interface/SimpleTransmission</type>
+     <joint name="l_arm_sh_p">
+       <hardwareInterface>EffortJointInterface</hardwareInterface>
+     </joint>
+     <actuator name="l_arm_sh_p_motor">
        <hardwareInterface>EffortJointInterface</hardwareInterface>
        <mechanicalReduction>1</mechanicalReduction>
@@ -84,18 +84,18 @@
   </link>
   <!-- left_arm_roll -->
- <joint name="l_arm_shoulder_roll" type="revolute">
+ <joint name="l_arm_sh_r" type="revolute">
     <parent link="l_arm_shoulder_pitch_link"/>
     <child link="l_arm_shoulder_roll_link"/>
     <origin xyz="0 0.097 0" rpy="0 0 0"/>
-    <axis xyz="0 1 0"/>
-    <limit velocity="6.5" effort="1000" lower="${-pi/2}" upper="${pi}" />
-    <dynamics damping = "0.7"/>
-  </joint>
-  <transmission name="l_arm_shoulder_roll_tran">
-     <type>transmission_interface/SimpleTransmission</type>
-     <joint name="l_arm_shoulder_roll">
-       <hardwareInterface>EffortJointInterface</hardwareInterface>
-     </joint>
-     <actuator name="l_arm_shoulder_roll_motor">
+    <axis xyz="1 0 0"/>
+    <limit velocity="6.5" effort="1000" lower="${-pi/2}" upper="${pi}" />
+    <dynamics damping = "0.7"/>
+  </joint>
+  <transmission name="l_arm_sh_r_tran">
+     <type>transmission_interface/SimpleTransmission</type>
+     <joint name="l_arm_sh_r">
+       <hardwareInterface>EffortJointInterface</hardwareInterface>
+     </joint>
+     <actuator name="l_arm_sh_r_motor">
        <hardwareInterface>EffortJointInterface</hardwareInterface>
        <mechanicalReduction>1</mechanicalReduction>
@@ -123,18 +123,18 @@
   </link>
   <!-- left_arm_yaw -->
-<joint name="l_arm_shoulder_yaw" type="revolute">
+<joint name="l_arm_sh_y" type="revolute">
     <parent link="l_arm_shoulder_roll_link"/>
     <child link="l_arm_shoulder_yaw_link"/>
     <origin xyz="0 0 -0.047" rpy="0 0 0"/>
-    <axis xyz="0 1 0"/>
-    <limit velocity="6.5" effort="1000" lower="${-pi/2}" upper="${pi}" />
-    <dynamics damping = "0.7"/>
-  </joint>
-  <transmission name="l_arm_shoulder_yaw_tran">
-     <type>transmission_interface/SimpleTransmission</type>
-     <joint name="l_arm_shoulder_yaw">
-       <hardwareInterface>EffortJointInterface</hardwareInterface>
-     </joint>
-     <actuator name="l_arm_shoulder_yaw_motor">
+    <axis xyz="0 0 1"/>
+    <limit velocity="6.5" effort="1000" lower="${-pi/2}" upper="${pi}" />
+    <dynamics damping = "0.7"/>
+  </joint>
+  <transmission name="l_arm_sh_y_tran">
+     <type>transmission_interface/SimpleTransmission</type>
+     <joint name="l_arm_sh_y">
+       <hardwareInterface>EffortJointInterface</hardwareInterface>
+     </joint>
+     <actuator name="l_arm_sh_y_motor">
        <hardwareInterface>EffortJointInterface</hardwareInterface>
        <mechanicalReduction>1</mechanicalReduction>
@@ -162,5 +162,5 @@
   </link>
   <!-- left_arm_elbow -->
-<joint name="l_arm_elbow_pitch" type="revolute">
+<joint name="l_arm_el_p" type="revolute">
     <parent link="l_arm_shoulder_yaw_link"/>
     <child link="l_arm_elbow_pitch_link"/>
@@ -170,10 +170,10 @@
     <dynamics damping = "0.7"/>
   </joint>
-  <transmission name="l_arm_elbow_pitch_tran">
-     <type>transmission_interface/SimpleTransmission</type>
-     <joint name="l_arm_elbow_pitch">
-       <hardwareInterface>EffortJointInterface</hardwareInterface>
-     </joint>
-     <actuator name="l_arm_elbow_pitch_motor">
+  <transmission name="l_arm_el_p_tran">
+     <type>transmission_interface/SimpleTransmission</type>
+     <joint name="l_arm_el_p">
+       <hardwareInterface>EffortJointInterface</hardwareInterface>
+     </joint>
+     <actuator name="l_arm_el_p_motor">
        <hardwareInterface>EffortJointInterface</hardwareInterface>
        <mechanicalReduction>1</mechanicalReduction>
@@ -201,5 +201,5 @@
   </link>
   <!-- left_arm_wrist_pitch -->
-<joint name="l_arm_wrist_pitch" type="revolute">
+<joint name="l_arm_wr_p" type="revolute">
     <parent link="l_arm_elbow_pitch_link"/>
     <child link="l_arm_wrist_pitch_link"/>
@@ -209,10 +209,10 @@
     <dynamics damping = "0.7"/>
   </joint>
-  <transmission name="l_arm_wrist_pitch_tran">
-     <type>transmission_interface/SimpleTransmission</type>
-     <joint name="l_arm_wrist_pitch">
-       <hardwareInterface>EffortJointInterface</hardwareInterface>
-     </joint>
-     <actuator name="l_arm_wrist_pitch_motor">
+  <transmission name="l_arm_wr_p_tran">
+     <type>transmission_interface/SimpleTransmission</type>
+     <joint name="l_arm_wr_p">
+       <hardwareInterface>EffortJointInterface</hardwareInterface>
+     </joint>
+     <actuator name="l_arm_wr_p_motor">
        <hardwareInterface>EffortJointInterface</hardwareInterface>
        <mechanicalReduction>1</mechanicalReduction>
@@ -240,18 +240,18 @@
   </link>
 <!-- left_arm_wrist_roll -->
-<joint name="l_arm_wrist_roll" type="revolute">
+<joint name="l_arm_wr_r" type="revolute">
     <parent link="l_arm_wrist_pitch_link"/>
     <child link="l_arm_wrist_roll_link"/>
     <origin xyz="0 0 0" rpy="0 0 0"/>
-    <axis xyz="0 1 0"/>
-    <limit velocity="6.5" effort="1000" lower="${-pi/2}" upper="${pi}" />
-    <dynamics damping = "0.7"/>
-  </joint>
-  <transmission name="l_arm_wrist_roll_tran">
-     <type>transmission_interface/SimpleTransmission</type>
-     <joint name="l_arm_wrist_roll">
-       <hardwareInterface>EffortJointInterface</hardwareInterface>
-     </joint>
-     <actuator name="l_arm_wrist_roll_motor">
+    <axis xyz="1 0 0"/>
+    <limit velocity="6.5" effort="1000" lower="${-pi/2}" upper="${pi}" />
+    <dynamics damping = "0.7"/>
+  </joint>
+  <transmission name="l_arm_wr_r_tran">
+     <type>transmission_interface/SimpleTransmission</type>
+     <joint name="l_arm_wr_r">
+       <hardwareInterface>EffortJointInterface</hardwareInterface>
+     </joint>
+     <actuator name="l_arm_wr_r_motor">
        <hardwareInterface>EffortJointInterface</hardwareInterface>
        <mechanicalReduction>1</mechanicalReduction>
@@ -280,5 +280,5 @@
     <!-- right_arm -->
   <!-- right_arm_pitch -->
- <joint name="r_arm_shoulder_pitch" type="revolute">
+ <joint name="r_arm_sh_p" type="revolute">
     <parent link="body_main"/>
     <child link="r_arm_shoulder_pitch_link"/>
@@ -288,10 +288,10 @@
     <dynamics damping = "0.7"/>
   </joint>
-  <transmission name="r_arm_shoulder_pitch_tran">
-     <type>transmission_interface/SimpleTransmission</type>
-     <joint name="r_arm_shoulder_pitch">
-       <hardwareInterface>EffortJointInterface</hardwareInterface>
-     </joint>
-     <actuator name="r_arm_shoulder_pitch_motor">
+  <transmission name="r_arm_sh_p_tran">
+     <type>transmission_interface/SimpleTransmission</type>
+     <joint name="r_arm_sh_p">
+       <hardwareInterface>EffortJointInterface</hardwareInterface>
+     </joint>
+     <actuator name="r_arm_sh_p_motor">
        <hardwareInterface>EffortJointInterface</hardwareInterface>
        <mechanicalReduction>1</mechanicalReduction>
@@ -319,18 +319,18 @@
   </link>
   <!-- right_arm_roll -->
- <joint name="r_arm_shoulder_roll" type="revolute">
+ <joint name="r_arm_sh_r" type="revolute">
     <parent link="r_arm_shoulder_pitch_link"/>
     <child link="r_arm_shoulder_roll_link"/>
     <origin xyz="0 -0.097 0" rpy="0 0 0"/>
-    <axis xyz="0 1 0"/>
-    <limit velocity="6.5" effort="1000" lower="${-pi/2}" upper="${pi}" />
-    <dynamics damping = "0.7"/>
-  </joint>
-  <transmission name="r_arm_shoulder_roll_tran">
-     <type>transmission_interface/SimpleTransmission</type>
-     <joint name="r_arm_shoulder_roll">
-       <hardwareInterface>EffortJointInterface</hardwareInterface>
-     </joint>
-     <actuator name="r_arm_shoulder_roll_motor">
+    <axis xyz="1 0 0"/>
+    <limit velocity="6.5" effort="1000" lower="${-pi/2}" upper="${pi}" />
+    <dynamics damping = "0.7"/>
+  </joint>
+  <transmission name="r_arm_sh_r_tran">
+     <type>transmission_interface/SimpleTransmission</type>
+     <joint name="r_arm_sh_r">
+       <hardwareInterface>EffortJointInterface</hardwareInterface>
+     </joint>
+     <actuator name="r_arm_sh_r_motor">
        <hardwareInterface>EffortJointInterface</hardwareInterface>
        <mechanicalReduction>1</mechanicalReduction>
@@ -358,18 +358,18 @@
   </link>
   <!-- right_arm_yaw -->
-<joint name="r_arm_shoulder_yaw" type="revolute">
+<joint name="r_arm_sh_y" type="revolute">
     <parent link="r_arm_shoulder_roll_link"/>
     <child link="r_arm_shoulder_yaw_link"/>
     <origin xyz="0 0 -0.047" rpy="0 0 0"/>
-    <axis xyz="0 1 0"/>
-    <limit velocity="6.5" effort="1000" lower="${-pi/2}" upper="${pi}" />
-    <dynamics damping = "0.7"/>
-  </joint>
-  <transmission name="r_arm_shoulder_yaw_tran">
-     <type>transmission_interface/SimpleTransmission</type>
-     <joint name="r_arm_shoulder_yaw">
-       <hardwareInterface>EffortJointInterface</hardwareInterface>
-     </joint>
-     <actuator name="r_arm_shoulder_yaw_motor">
+    <axis xyz="0 0 1"/>
+    <limit velocity="6.5" effort="1000" lower="${-pi/2}" upper="${pi}" />
+    <dynamics damping = "0.7"/>
+  </joint>
+  <transmission name="r_arm_sh_y_tran">
+     <type>transmission_interface/SimpleTransmission</type>
+     <joint name="r_arm_sh_y">
+       <hardwareInterface>EffortJointInterface</hardwareInterface>
+     </joint>
+     <actuator name="r_arm_sh_y_motor">
        <hardwareInterface>EffortJointInterface</hardwareInterface>
        <mechanicalReduction>1</mechanicalReduction>
@@ -397,5 +397,5 @@
   </link>
   <!-- right_arm_elbow -->
-<joint name="r_arm_elbow_pitch" type="revolute">
+<joint name="r_arm_el_p" type="revolute">
     <parent link="r_arm_shoulder_yaw_link"/>
     <child link="r_arm_elbow_pitch_link"/>
@@ -405,10 +405,10 @@
     <dynamics damping = "0.7"/>
   </joint>
-  <transmission name="r_arm_elbow_pitch_tran">
-     <type>transmission_interface/SimpleTransmission</type>
-     <joint name="r_arm_elbow_pitch">
-       <hardwareInterface>EffortJointInterface</hardwareInterface>
-     </joint>
-     <actuator name="r_arm_elbow_pitch_motor">
+  <transmission name="r_arm_el_p_tran">
+     <type>transmission_interface/SimpleTransmission</type>
+     <joint name="r_arm_el_p">
+       <hardwareInterface>EffortJointInterface</hardwareInterface>
+     </joint>
+     <actuator name="r_arm_el_p_motor">
        <hardwareInterface>EffortJointInterface</hardwareInterface>
        <mechanicalReduction>1</mechanicalReduction>
@@ -436,5 +436,5 @@
   </link>
   <!-- right_arm_wrist_pitch -->
-<joint name="r_arm_wrist_pitch" type="revolute">
+<joint name="r_arm_wr_p" type="revolute">
     <parent link="r_arm_elbow_pitch_link"/>
     <child link="r_arm_wrist_pitch_link"/>
@@ -444,10 +444,10 @@
     <dynamics damping = "0.7"/>
   </joint>
-  <transmission name="r_arm_wrist_pitch_tran">
-     <type>transmission_interface/SimpleTransmission</type>
-     <joint name="r_arm_wrist_pitch">
-       <hardwareInterface>EffortJointInterface</hardwareInterface>
-     </joint>
-     <actuator name="r_arm_wrist_pitch_motor">
+  <transmission name="r_arm_wr_p_tran">
+     <type>transmission_interface/SimpleTransmission</type>
+     <joint name="r_arm_wr_p">
+       <hardwareInterface>EffortJointInterface</hardwareInterface>
+     </joint>
+     <actuator name="r_arm_wr_p_motor">
        <hardwareInterface>EffortJointInterface</hardwareInterface>
        <mechanicalReduction>1</mechanicalReduction>
@@ -475,18 +475,18 @@
   </link>
 <!-- right_arm_wrist_roll -->
-<joint name="r_arm_wrist_roll" type="revolute">
+<joint name="r_arm_wr_r" type="revolute">
     <parent link="r_arm_wrist_pitch_link"/>
     <child link="r_arm_wrist_roll_link"/>
     <origin xyz="0 0 0" rpy="0 0 0"/>
-    <axis xyz="0 1 0"/>
-    <limit velocity="6.5" effort="1000" lower="${-pi/2}" upper="${pi}" />
-    <dynamics damping = "0.7"/>
-  </joint>
-  <transmission name="r_arm_wrist_roll_tran">
-     <type>transmission_interface/SimpleTransmission</type>
-     <joint name="r_arm_wrist_roll">
-       <hardwareInterface>EffortJointInterface</hardwareInterface>
-     </joint>
-     <actuator name="r_arm_wrist_roll_motor">
+    <axis xyz="1 0 0"/>
+    <limit velocity="6.5" effort="1000" lower="${-pi/2}" upper="${pi}" />
+    <dynamics damping = "0.7"/>
+  </joint>
+  <transmission name="r_arm_wr_r_tran">
+     <type>transmission_interface/SimpleTransmission</type>
+     <joint name="r_arm_wr_r">
+       <hardwareInterface>EffortJointInterface</hardwareInterface>
+     </joint>
+     <actuator name="r_arm_wr_r_motor">
        <hardwareInterface>EffortJointInterface</hardwareInterface>
        <mechanicalReduction>1</mechanicalReduction>

Commit message: gazebo model modified

File: erica_description/urdf/erica_robot.xacro (robot description, xacro)
@@ -18,5 +18,5 @@
   </link>
   <joint name="base_fixed" type="fixed">
-    <origin xyz="0 0 0.9" rpy="0 0 0"/>
+    <origin xyz="0 0 1" rpy="0 0 0"/>
     <parent link="base"/>
     <child link="body_main"/>
@@ -39,5 +39,5 @@
     <inertial>
       <origin xyz="0 0 0" rpy="0 0 0"/>
-      <mass value="1"/>
+      <mass value="100"/>
       <inertia ixx="1.0" ixy="0.0" ixz="0.0" iyy="1.0" iyz="0.0" izz="1.0" />
     </inertial>
@@ -88,5 +88,5 @@
     <child link="l_arm_shoulder_roll_link"/>
     <origin xyz="0 0.097 0" rpy="0 0 0"/>
-    <axis xyz="1 0 0"/>
+    <axis xyz="0 0 -1"/>
     <limit velocity="6.5" effort="1000" lower="${-pi/2}" upper="${pi}" />
     <dynamics damping = "0.7"/>
@@ -126,6 +126,6 @@
     <parent link="l_arm_shoulder_roll_link"/>
     <child link="l_arm_shoulder_yaw_link"/>
-    <origin xyz="0 0 -0.047" rpy="0 0 0"/>
-    <axis xyz="0 0 1"/>
+    <origin xyz="0.047 0 0" rpy="0 0 0"/>
+    <axis xyz="-1 0 0"/>
     <limit velocity="6.5" effort="1000" lower="${-pi/2}" upper="${pi}" />
     <dynamics damping = "0.7"/>
@@ -165,6 +165,6 @@
     <parent link="l_arm_shoulder_yaw_link"/>
     <child link="l_arm_elbow_pitch_link"/>
-    <origin xyz="0 0 -0.153" rpy="0 0 0"/>
-    <axis xyz="0 1 0"/>
+    <origin xyz="0.153 0 0" rpy="0 0 0"/>
+    <axis xyz="0 -1 0"/>
     <limit velocity="6.5" effort="1000" lower="${-pi/2}" upper="${pi}" />
     <dynamics damping = "0.7"/>
@@ -204,6 +204,6 @@
     <parent link="l_arm_elbow_pitch_link"/>
     <child link="l_arm_wrist_pitch_link"/>
-    <origin xyz="0 0 -0.2" rpy="0 0 0"/>
-    <axis xyz="0 1 0"/>
+    <origin xyz="0.2 0 0" rpy="0 0 0"/>
+    <axis xyz="0 -1 0"/>
     <limit velocity="6.5" effort="1000" lower="${-pi/2}" upper="${pi}" />
     <dynamics damping = "0.7"/>
@@ -244,5 +244,5 @@
     <child link="l_arm_wrist_roll_link"/>
     <origin xyz="0 0 0" rpy="0 0 0"/>
-    <axis xyz="1 0 0"/>
+    <axis xyz="0 0 -1"/>
     <limit velocity="6.5" effort="1000" lower="${-pi/2}" upper="${pi}" />
     <dynamics damping = "0.7"/>
@@ -284,5 +284,5 @@
     <child link="r_arm_shoulder_pitch_link"/>
     <origin xyz="0 -0.113 0" rpy="0 0 0"/>
-    <axis xyz="0 1 0"/>
+    <axis xyz="0 -1 0"/>
     <limit velocity="6.5" effort="1000" lower="${-pi/2}" upper="${pi}" />
     <dynamics damping = "0.7"/>
@@ -323,5 +323,5 @@
     <child link="r_arm_shoulder_roll_link"/>
     <origin xyz="0 -0.097 0" rpy="0 0 0"/>
-    <axis xyz="1 0 0"/>
+    <axis xyz="0 0 -1"/>
     <limit velocity="6.5" effort="1000" lower="${-pi/2}" upper="${pi}" />
     <dynamics damping = "0.7"/>
@@ -361,6 +361,6 @@
     <parent link="r_arm_shoulder_roll_link"/>
     <child link="r_arm_shoulder_yaw_link"/>
-    <origin xyz="0 0 -0.047" rpy="0 0 0"/>
-    <axis xyz="0 0 1"/>
+    <origin xyz="0.047 0 0" rpy="0 0 0"/>
+    <axis xyz="-1 0 0"/>
     <limit velocity="6.5" effort="1000" lower="${-pi/2}" upper="${pi}" />
     <dynamics damping = "0.7"/>
@@ -400,5 +400,5 @@
     <parent link="r_arm_shoulder_yaw_link"/>
     <child link="r_arm_elbow_pitch_link"/>
-    <origin xyz="0 0 -0.153" rpy="0 0 0"/>
+    <origin xyz="0.153 0 0" rpy="0 0 0"/>
     <axis xyz="0 1 0"/>
     <limit velocity="6.5" effort="1000" lower="${-pi/2}" upper="${pi}" />
@@ -439,5 +439,5 @@
     <parent link="r_arm_elbow_pitch_link"/>
     <child link="r_arm_wrist_pitch_link"/>
-    <origin xyz="0 0 -0.2" rpy="0 0 0"/>
+    <origin xyz="0.2 0 0" rpy="0 0 0"/>
     <axis xyz="0 1 0"/>
     <limit velocity="6.5" effort="1000" lower="${-pi/2}" upper="${pi}" />
@@ -479,5 +479,5 @@
     <child link="r_arm_wrist_roll_link"/>
     <origin xyz="0 0 0" rpy="0 0 0"/>
-    <axis xyz="1 0 0"/>
+    <axis xyz="0 0 -1"/>
     <limit velocity="6.5" effort="1000" lower="${-pi/2}" upper="${pi}" />
     <dynamics damping = "0.7"/>

Commit message: m

File: erica_description/urdf/erica_robot.xacro (robot description, xacro)
@@ -35,5 +35,5 @@
           <mesh filename="package://erica_description/meshes/asm_don_big_main.stl" scale="0.001 0.001 0.001"/>
         </geometry>
-        <material name="red"/>
+        <material name="white"/>
     </visual>
     <inertial>
@@ -75,5 +75,5 @@
           <mesh filename="package://erica_description/meshes/asm_don_big_arm_l-1.stl" scale="0.001 0.001 0.001"/>
         </geometry>
-        <material name="red"/>
+        <material name="white"/>
     </visual>
     <inertial>
@@ -114,5 +114,5 @@
           <mesh filename="package://erica_description/meshes/asm_don_big_arm_l-2.stl" scale="0.001 0.001 0.001"/>
         </geometry>
-        <material name="red"/>
+        <material name="white"/>
     </visual>
     <inertial>
@@ -153,5 +153,5 @@
           <mesh filename="package://erica_description/meshes/asm_don_big_arm_l-3.stl" scale="0.001 0.001 0.001"/>
         </geometry>
-        <material name="red"/>
+        <material name="white"/>
     </visual>
     <inertial>
@@ -192,5 +192,5 @@
           <mesh filename="package://erica_description/meshes/asm_don_big_arm_l-4.stl" scale="0.001 0.001 0.001"/>
         </geometry>
-        <material name="red"/>
+        <material name="white"/>
     </visual>
     <inertial>
@@ -231,5 +231,5 @@
           <mesh filename="package://erica_description/meshes/asm_don_big_arm_l-5.stl" scale="0.001 0.001 0.001"/>
         </geometry>
-        <material name="red"/>
+        <material name="white"/>
     </visual>
     <inertial>
@@ -270,5 +270,5 @@
           <mesh filename="package://erica_description/meshes/asm_don_big_arm_l-6.stl" scale="0.001 0.001 0.001"/>
         </geometry>
-        <material name="red"/>
+        <material name="white"/>
     </visual>
     <inertial>
@@ -310,5 +310,5 @@
           <mesh filename="package://erica_description/meshes/asm_don_big_arm_r-1.stl" scale="0.001 0.001 0.001"/>
         </geometry>
-        <material name="red"/>
+        <material name="white"/>
     </visual>
     <inertial>
@@ -349,5 +349,5 @@
           <mesh filename="package://erica_description/meshes/asm_don_big_arm_r-2.stl" scale="0.001 0.001 0.001"/>
         </geometry>
-        <material name="red"/>
+        <material name="white"/>
     </visual>
     <inertial>
@@ -388,5 +388,5 @@
           <mesh filename="package://erica_description/meshes/asm_don_big_arm_r-3.stl" scale="0.001 0.001 0.001"/>
         </geometry>
-        <material name="red"/>
+        <material name="white"/>
     </visual>
     <inertial>
@@ -427,5 +427,5 @@
           <mesh filename="package://erica_description/meshes/asm_don_big_arm_r-4.stl" scale="0.001 0.001 0.001"/>
         </geometry>
-        <material name="red"/>
+        <material name="white"/>
     </visual>
     <inertial>
@@ -466,5 +466,5 @@
           <mesh filename="package://erica_description/meshes/asm_don_big_arm_r-5.stl" scale="0.001 0.001 0.001"/>
         </geometry>
-        <material name="red"/>
+        <material name="white"/>
     </visual>
     <inertial>
@@ -505,5 +505,5 @@
           <mesh filename="package://erica_description/meshes/asm_don_big_arm_r-6.stl" scale="0.001 0.001 0.001"/>
         </geometry>
-        <material name="red"/>
+        <material name="white"/>
     </visual>
     <inertial>

Commit message: add zed links to urdf and change rviz setting

File: erica_description/urdf/erica_robot.xacro (robot description, xacro)
@@ -43,4 +43,38 @@
     </inertial>
   </link>
+  <!-- head(zed) -->
+   <joint name="camera_joint" type="fixed">
+    <parent link="body_main"/>
+    <child link="zed_camera_center"/>
+    <origin xyz="0 0 0.195" rpy="0 0 0"/>
+  </joint>
+  <!-- Camera Center -->
+  <link name="zed_camera_center"/>
+  <!-- Left Camera -->
+    <joint name="zed_left_camera_joint" type="fixed">
+        <parent link="zed_camera_center"/>
+        <child link="zed_left_camera_frame"/>
+        <origin xyz="0 0.06 0" rpy="0 0 0" />
+    </joint>
+    <link name="zed_left_camera_frame" />
+    <joint name="zed_left_camera_optical_joint" type="fixed">
+        <origin xyz="0 0 0" rpy="-1.57079632679 0.0 -1.57079632679"/>
+        <parent link="zed_left_camera_frame"/>
+        <child link="zed_left_camera_optical_frame"/>
+    </joint>
+    <link name="zed_left_camera_optical_frame"/>
+  <!-- Right Camera -->
+    <joint name="zed_right_camera_joint" type="fixed">
+        <parent link="zed_camera_center"/>
+        <child link="zed_right_camera_frame"/>
+        <origin xyz="0 -0.06 0" rpy="0 0 0" />
+    </joint>
+    <link name="zed_right_camera_frame" />
+    <joint name="zed_right_camera_optical_joint" type="fixed">
+        <origin xyz="0 0 0" rpy="-1.57079632679 0.0 -1.57079632679"/>
+        <parent link="zed_right_camera_frame"/>
+        <child link="zed_right_camera_optical_frame"/>
+    </joint>
+    <link name="zed_right_camera_optical_frame"/>
   <!-- left_arm -->
   <!-- left_arm_pitch -->
