Commit message: change zed link position slightly

File: erica_description/urdf/erica_robot.xacro (robot description, xacro)
@@ -47,37 +47,37 @@
     <parent link="body_main"/>
     <child link="zed_camera_center"/>
-    <origin xyz="0 0 0.195" rpy="0 0 0"/>
+    <origin xyz="0.09 0 0.195" rpy="0 0 0"/>
   </joint>
   <!-- Camera Center -->
   <link name="zed_camera_center"/>
   <!-- Left Camera -->
-    <joint name="zed_left_camera_joint" type="fixed">
-        <parent link="zed_camera_center"/>
-        <child link="zed_left_camera_frame"/>
-        <origin xyz="0 0.06 0" rpy="0 0 0" />
-    </joint>
+  <joint name="zed_left_camera_joint" type="fixed">
+   <parent link="zed_camera_center"/>
+   <child link="zed_left_camera_frame"/>
+   <origin xyz="0 0.06 0" rpy="0 0 0" />
+  </joint>
     <link name="zed_left_camera_frame" />
-    <joint name="zed_left_camera_optical_joint" type="fixed">
-        <origin xyz="0 0 0" rpy="-1.57079632679 0.0 -1.57079632679"/>
-        <parent link="zed_left_camera_frame"/>
-        <child link="zed_left_camera_optical_frame"/>
-    </joint>
-    <link name="zed_left_camera_optical_frame"/>
+  <joint name="zed_left_camera_optical_joint" type="fixed">
+    <origin xyz="0 0 0" rpy="-1.57079632679 0.0 -1.57079632679"/>
+    <parent link="zed_left_camera_frame"/>
+    <child link="zed_left_camera_optical_frame"/>
+  </joint>
+  <link name="zed_left_camera_optical_frame"/>
   <!-- Right Camera -->
-    <joint name="zed_right_camera_joint" type="fixed">
-        <parent link="zed_camera_center"/>
-        <child link="zed_right_camera_frame"/>
-        <origin xyz="0 -0.06 0" rpy="0 0 0" />
-    </joint>
-    <link name="zed_right_camera_frame" />
-    <joint name="zed_right_camera_optical_joint" type="fixed">
-        <origin xyz="0 0 0" rpy="-1.57079632679 0.0 -1.57079632679"/>
-        <parent link="zed_right_camera_frame"/>
-        <child link="zed_right_camera_optical_frame"/>
-    </joint>
-    <link name="zed_right_camera_optical_frame"/>
+  <joint name="zed_right_camera_joint" type="fixed">
+    <parent link="zed_camera_center"/>
+    <child link="zed_right_camera_frame"/>
+    <origin xyz="0 -0.06 0" rpy="0 0 0" />
+  </joint>
+  <link name="zed_right_camera_frame" />
+  <joint name="zed_right_camera_optical_joint" type="fixed">
+   <origin xyz="0 0 0" rpy="-1.57079632679 0.0 -1.57079632679"/>
+   <parent link="zed_right_camera_frame"/>
+   <child link="zed_right_camera_optical_frame"/>
+  </joint>
+  <link name="zed_right_camera_optical_frame"/>
   <!-- left_arm -->
   <!-- left_arm_pitch -->
- <joint name="l_arm_sh_p" type="revolute">
+  <joint name="l_arm_sh_p" type="revolute">
     <parent link="body_main"/>
     <child link="l_arm_shoulder_pitch_link"/>

Commit message: modify joint limits in urdf

File: erica_description/urdf/erica_robot.xacro (robot description, xacro)
@@ -1,5 +1,5 @@
 <?xml version="1.0"?>
 <robot name="erica_robot" xmlns:xacro="http://www.ros.org/wiki/xacro">
-  <xacro:property name="pi" value="3.141592654" />
+  <xacro:property name="pi" value="3.14" />
    <!-- Import all Gazebo-customization elements, including Gazebo colors -->
   <xacro:include filename="$(find erica_description)/urdf/erica_gazebo.gazebo" />
@@ -39,5 +39,5 @@
     <inertial>
       <origin xyz="0 0 0" rpy="0 0 0"/>
-      <mass value="100"/>
+      <mass value="300"/>
       <inertia ixx="1.0" ixy="0.0" ixz="0.0" iyy="1.0" iyz="0.0" izz="1.0" />
     </inertial>
@@ -84,5 +84,5 @@
     <origin xyz="0 0.113 0" rpy="0 0 0"/>
     <axis xyz="0 1 0"/>
-    <limit velocity="6.5" effort="1000" lower="${-pi/2}" upper="${pi}" />
+    <limit velocity="6.5" effort="1000" lower="${-pi}" upper="${pi}" />
     <dynamics damping = "0.7"/>
   </joint>
@@ -123,5 +123,5 @@
     <origin xyz="0 0.097 0" rpy="0 0 0"/>
     <axis xyz="0 0 -1"/>
-    <limit velocity="6.5" effort="1000" lower="${-pi/2}" upper="${pi}" />
+    <limit velocity="6.5" effort="1000" lower="${-pi}" upper="${pi}" />
     <dynamics damping = "0.7"/>
   </joint>
@@ -162,5 +162,5 @@
     <origin xyz="0.047 0 0" rpy="0 0 0"/>
     <axis xyz="-1 0 0"/>
-    <limit velocity="6.5" effort="1000" lower="${-pi/2}" upper="${pi}" />
+    <limit velocity="6.5" effort="1000" lower="${-pi}" upper="${pi}" />
     <dynamics damping = "0.7"/>
   </joint>
@@ -201,5 +201,5 @@
     <origin xyz="0.153 0 0" rpy="0 0 0"/>
     <axis xyz="0 -1 0"/>
-    <limit velocity="6.5" effort="1000" lower="${-pi/2}" upper="${pi}" />
+    <limit velocity="6.5" effort="1000" lower="${-pi}" upper="${pi}" />
     <dynamics damping = "0.7"/>
   </joint>
@@ -240,5 +240,5 @@
     <origin xyz="0.2 0 0" rpy="0 0 0"/>
     <axis xyz="0 -1 0"/>
-    <limit velocity="6.5" effort="1000" lower="${-pi/2}" upper="${pi}" />
+    <limit velocity="6.5" effort="1000" lower="${-pi}" upper="${pi}" />
     <dynamics damping = "0.7"/>
   </joint>
@@ -279,5 +279,5 @@
     <origin xyz="0 0 0" rpy="0 0 0"/>
     <axis xyz="0 0 -1"/>
-    <limit velocity="6.5" effort="1000" lower="${-pi/2}" upper="${pi}" />
+    <limit velocity="6.5" effort="1000" lower="${-pi}" upper="${pi}" />
     <dynamics damping = "0.7"/>
   </joint>
@@ -319,5 +319,5 @@
     <origin xyz="0 -0.113 0" rpy="0 0 0"/>
     <axis xyz="0 -1 0"/>
-    <limit velocity="6.5" effort="1000" lower="${-pi/2}" upper="${pi}" />
+    <limit velocity="6.5" effort="1000" lower="${-pi}" upper="${pi}" />
     <dynamics damping = "0.7"/>
   </joint>
@@ -358,5 +358,5 @@
     <origin xyz="0 -0.097 0" rpy="0 0 0"/>
     <axis xyz="0 0 -1"/>
-    <limit velocity="6.5" effort="1000" lower="${-pi/2}" upper="${pi}" />
+    <limit velocity="6.5" effort="1000" lower="${-pi}" upper="${pi}" />
     <dynamics damping = "0.7"/>
   </joint>
@@ -397,5 +397,5 @@
     <origin xyz="0.047 0 0" rpy="0 0 0"/>
     <axis xyz="-1 0 0"/>
-    <limit velocity="6.5" effort="1000" lower="${-pi/2}" upper="${pi}" />
+    <limit velocity="6.5" effort="1000" lower="${-pi}" upper="${pi}" />
     <dynamics damping = "0.7"/>
   </joint>
@@ -436,5 +436,5 @@
     <origin xyz="0.153 0 0" rpy="0 0 0"/>
     <axis xyz="0 1 0"/>
-    <limit velocity="6.5" effort="1000" lower="${-pi/2}" upper="${pi}" />
+    <limit velocity="6.5" effort="1000" lower="${-pi}" upper="${pi}" />
     <dynamics damping = "0.7"/>
   </joint>
@@ -475,5 +475,5 @@
     <origin xyz="0.2 0 0" rpy="0 0 0"/>
     <axis xyz="0 1 0"/>
-    <limit velocity="6.5" effort="1000" lower="${-pi/2}" upper="${pi}" />
+    <limit velocity="6.5" effort="1000" lower="${-pi}" upper="${pi}" />
     <dynamics damping = "0.7"/>
   </joint>
@@ -514,5 +514,5 @@
     <origin xyz="0 0 0" rpy="0 0 0"/>
     <axis xyz="0 0 -1"/>
-    <limit velocity="6.5" effort="1000" lower="${-pi/2}" upper="${pi}" />
+    <limit velocity="6.5" effort="1000" lower="${-pi}" upper="${pi}" />
     <dynamics damping = "0.7"/>
   </joint>

Commit message: modified

File: erica_description/urdf/erica_robot.xacro (robot description, xacro)
@@ -27,11 +27,11 @@
       <origin xyz="0 0 0" rpy="0 0 0"/>
          <geometry>
-          <mesh filename="package://erica_description/meshes/asm_don_big_main.stl" scale="0.001 0.001 0.001"/>
-        </geometry>
-    </collision>
-    <visual>
-        <origin xyz="0 0 0" rpy="0 0 0"/>
-        <geometry>
-          <mesh filename="package://erica_description/meshes/asm_don_big_main.stl" scale="0.001 0.001 0.001"/>
+          <mesh filename="package://erica_description/meshes/prt_gazevo_test.stl" scale="1 1 1"/>
+        </geometry>
+    </collision>
+    <visual>
+        <origin xyz="0 0 0" rpy="0 0 0"/>
+        <geometry>
+          <mesh filename="package://erica_description/meshes/prt_gazevo_test.stl" scale="1 1 1"/>
         </geometry>
         <material name="white"/>

Commit message: model completed

File: erica_description/urdf/erica_robot.xacro (robot description, xacro)
@@ -14,12 +14,12 @@
     <child link="pelvis"/>
   </joint>
--->
   <link name="base">
   </link>
   <joint name="base_fixed" type="fixed">
-    <origin xyz="0 0 1" rpy="0 0 0"/>
+    <origin xyz="0 0 0.2" rpy="0 0 0"/>
     <parent link="base"/>
     <child link="body_main"/>
   </joint>
+-->
   <!-- main -->
  <link name="body_main">
@@ -27,11 +27,11 @@
       <origin xyz="0 0 0" rpy="0 0 0"/>
          <geometry>
-          <mesh filename="package://erica_description/meshes/prt_gazevo_test.stl" scale="1 1 1"/>
-        </geometry>
-    </collision>
-    <visual>
-        <origin xyz="0 0 0" rpy="0 0 0"/>
-        <geometry>
-          <mesh filename="package://erica_description/meshes/prt_gazevo_test.stl" scale="1 1 1"/>
+          <mesh filename="package://erica_description/meshes/asm_don_big_main.stl" scale="0.001 0.001 0.001"/>
+        </geometry>
+    </collision>
+    <visual>
+        <origin xyz="0 0 0" rpy="0 0 0"/>
+        <geometry>
+          <mesh filename="package://erica_description/meshes/asm_don_big_main.stl" scale="0.001 0.001 0.001"/>
         </geometry>
         <material name="white"/>
@@ -40,4 +40,303 @@
       <origin xyz="0 0 0" rpy="0 0 0"/>
       <mass value="300"/>
+      <inertia ixx="1.0" ixy="0.0" ixz="0.0" iyy="1.0" iyz="0.0" izz="1.0" />
+    </inertial>
+  </link>
+  <!-- left wheel front-->
+  <joint name="left_wheel_front_joint" type="revolute">
+    <origin xyz="0.09 0.157 0.037" rpy="0 0 0"/>
+    <parent link="body_main"/>
+    <child link="left_wheel_front"/>
+    <axis xyz="0 1 0"/>
+    <limit velocity="6.5" effort="1000" lower="${-pi}" upper="${pi}" />
+    <dynamics damping = "0.7"/>
+  </joint>
+<transmission name="left_wheel_front_joint_tran">
+     <type>transmission_interface/SimpleTransmission</type>
+     <joint name="left_wheel_front_joint">
+       <hardwareInterface>EffortJointInterface</hardwareInterface>
+     </joint>
+     <actuator name="left_wheel_front_joint_motor">
+       <hardwareInterface>EffortJointInterface</hardwareInterface>
+       <mechanicalReduction>1</mechanicalReduction>
+     </actuator>
+  </transmission>
+ <link name="left_wheel_front">
+    <collision>
+      <origin xyz="0 0 0" rpy="0 0 0"/>
+         <geometry>
+          <mesh filename="package://erica_description/meshes/left_wheel_front.stl" scale="0.001 0.001 0.001"/>
+        </geometry>
+    </collision>
+    <visual>
+        <origin xyz="0 0 0" rpy="0 0 0"/>
+        <geometry>
+          <mesh filename="package://erica_description/meshes/left_wheel_front.stl" scale="0.001 0.001 0.001"/>
+        </geometry>
+        <material name="white"/>
+    </visual>
+    <inertial>
+      <origin xyz="0 0 0" rpy="0 0 0"/>
+      <mass value="1"/>
+      <inertia ixx="1.0" ixy="0.0" ixz="0.0" iyy="1.0" iyz="0.0" izz="1.0" />
+    </inertial>
+  </link>
+ <!-- right wheel front -->
+  <joint name="right_wheel_front_joint" type="revolute">
+    <origin xyz="0.09 -0.157 0.037" rpy="0 0 0"/>
+    <parent link="body_main"/>
+    <child link="right_wheel_front"/>
+    <axis xyz="0 1 0"/>
+    <limit velocity="6.5" effort="1000" lower="${-pi}" upper="${pi}" />
+    <dynamics damping = "0.7"/>
+  </joint>
+<transmission name="right_wheel_front_joint_tran">
+     <type>transmission_interface/SimpleTransmission</type>
+     <joint name="right_wheel_front_joint">
+       <hardwareInterface>EffortJointInterface</hardwareInterface>
+     </joint>
+     <actuator name="right_wheel_front_joint_motor">
+       <hardwareInterface>EffortJointInterface</hardwareInterface>
+       <mechanicalReduction>1</mechanicalReduction>
+     </actuator>
+  </transmission>
+ <link name="right_wheel_front">
+    <collision>
+      <origin xyz="0 0 0" rpy="0 0 0"/>
+         <geometry>
+          <mesh filename="package://erica_description/meshes/right_wheel_front.stl" scale="0.001 0.001 0.001"/>
+        </geometry>
+    </collision>
+    <visual>
+        <origin xyz="0 0 0" rpy="0 0 0"/>
+        <geometry>
+          <mesh filename="package://erica_description/meshes/right_wheel_front.stl" scale="0.001 0.001 0.001"/>
+        </geometry>
+        <material name="white"/>
+    </visual>
+    <inertial>
+      <origin xyz="0 0 0" rpy="0 0 0"/>
+      <mass value="1"/>
+      <inertia ixx="1.0" ixy="0.0" ixz="0.0" iyy="1.0" iyz="0.0" izz="1.0" />
+    </inertial>
+  </link>
+  <!-- left wheel rear-->
+  <joint name="left_wheel_rear_joint" type="revolute">
+    <origin xyz="-0.09 0.157 0.037" rpy="0 0 0"/>
+    <parent link="body_main"/>
+    <child link="left_wheel_rear"/>
+    <axis xyz="0 1 0"/>
+    <limit velocity="6.5" effort="1000" lower="${-pi}" upper="${pi}" />
+    <dynamics damping = "0.7"/>
+  </joint>
+<transmission name="left_wheel_rear_joint_tran">
+     <type>transmission_interface/SimpleTransmission</type>
+     <joint name="left_wheel_rear_joint">
+       <hardwareInterface>EffortJointInterface</hardwareInterface>
+     </joint>
+     <actuator name="left_wheel_rear_joint_motor">
+       <hardwareInterface>EffortJointInterface</hardwareInterface>
+       <mechanicalReduction>1</mechanicalReduction>
+     </actuator>
+  </transmission>
+ <link name="left_wheel_rear">
+    <collision>
+      <origin xyz="0 0 0" rpy="0 0 0"/>
+         <geometry>
+          <mesh filename="package://erica_description/meshes/left_wheel_rear.stl" scale="0.001 0.001 0.001"/>
+        </geometry>
+    </collision>
+    <visual>
+        <origin xyz="0 0 0" rpy="0 0 0"/>
+        <geometry>
+          <mesh filename="package://erica_description/meshes/left_wheel_rear.stl" scale="0.001 0.001 0.001"/>
+        </geometry>
+        <material name="white"/>
+    </visual>
+    <inertial>
+      <origin xyz="0 0 0" rpy="0 0 0"/>
+      <mass value="1"/>
+      <inertia ixx="1.0" ixy="0.0" ixz="0.0" iyy="1.0" iyz="0.0" izz="1.0" />
+    </inertial>
+  </link>
+ <!-- right wheel rear -->
+  <joint name="right_wheel_rear_joint" type="revolute">
+    <origin xyz="-0.09 -0.157 0.037" rpy="0 0 0"/>
+    <parent link="body_main"/>
+    <child link="right_wheel_rear"/>
+    <axis xyz="0 1 0"/>
+    <limit velocity="6.5" effort="1000" lower="${-pi}" upper="${pi}" />
+    <dynamics damping = "0.7"/>
+  </joint>
+<transmission name="right_wheel_rear_joint_tran">
+     <type>transmission_interface/SimpleTransmission</type>
+     <joint name="right_wheel_rear_joint">
+       <hardwareInterface>EffortJointInterface</hardwareInterface>
+     </joint>
+     <actuator name="right_wheel_rear_joint_motor">
+       <hardwareInterface>EffortJointInterface</hardwareInterface>
+       <mechanicalReduction>1</mechanicalReduction>
+     </actuator>
+  </transmission>
+ <link name="right_wheel_rear">
+    <collision>
+      <origin xyz="0 0 0" rpy="0 0 0"/>
+         <geometry>
+          <mesh filename="package://erica_description/meshes/right_wheel_rear.stl" scale="0.001 0.001 0.001"/>
+        </geometry>
+    </collision>
+    <visual>
+        <origin xyz="0 0 0" rpy="0 0 0"/>
+        <geometry>
+          <mesh filename="package://erica_description/meshes/right_wheel_rear.stl" scale="0.001 0.001 0.001"/>
+        </geometry>
+        <material name="white"/>
+    </visual>
+    <inertial>
+      <origin xyz="0 0 0" rpy="0 0 0"/>
+      <mass value="1"/>
+      <inertia ixx="1.0" ixy="0.0" ixz="0.0" iyy="1.0" iyz="0.0" izz="1.0" />
+    </inertial>
+  </link>
+<!-- neck-->
+  <joint name="neck_fixed_joint" type="fixed">
+    <origin xyz="0 0 0.933" rpy="0 0 0"/>
+    <parent link="body_main"/>
+    <child link="neck_joint"/>
+  </joint>
+ <link name="neck_joint">
+    <collision>
+      <origin xyz="0 0 0" rpy="0 0 0"/>
+         <geometry>
+          <mesh filename="package://erica_description/meshes/asm_don_big_neck.stl" scale="0.001 0.001 0.001"/>
+        </geometry>
+    </collision>
+    <visual>
+        <origin xyz="0 0 0" rpy="0 0 0"/>
+        <geometry>
+          <mesh filename="package://erica_description/meshes/asm_don_big_neck.stl" scale="0.001 0.001 0.001"/>
+        </geometry>
+        <material name="white"/>
+    </visual>
+    <inertial>
+      <origin xyz="0 0 0" rpy="0 0 0"/>
+      <mass value="1"/>
+      <inertia ixx="1.0" ixy="0.0" ixz="0.0" iyy="1.0" iyz="0.0" izz="1.0" />
+    </inertial>
+  </link>
+<!-- head_yaw -->
+  <joint name="head_yaw_joint" type="revolute">
+    <origin xyz="0 0 0.164" rpy="0 0 0"/>
+    <parent link="neck_joint"/>
+    <child link="head_yaw"/>
+    <axis xyz="0 0 1"/>
+    <limit velocity="6.5" effort="1000" lower="${-pi}" upper="${pi}" />
+    <dynamics damping = "0.7"/>
+  </joint>
+<transmission name="head_yaw_joint_tran">
+     <type>transmission_interface/SimpleTransmission</type>
+     <joint name="head_yaw_joint">
+       <hardwareInterface>EffortJointInterface</hardwareInterface>
+     </joint>
+     <actuator name="head_yaw_joint_motor">
+       <hardwareInterface>EffortJointInterface</hardwareInterface>
+       <mechanicalReduction>1</mechanicalReduction>
+     </actuator>
+  </transmission>
+ <link name="head_yaw">
+    <collision>
+      <origin xyz="0 0 0" rpy="0 0 0"/>
+         <geometry>
+          <mesh filename="package://erica_description/meshes/asm_don_big_main_head_yaw.stl" scale="0.001 0.001 0.001"/>
+        </geometry>
+    </collision>
+    <visual>
+        <origin xyz="0 0 0" rpy="0 0 0"/>
+        <geometry>
+          <mesh filename="package://erica_description/meshes/asm_don_big_main_head_yaw.stl" scale="0.001 0.001 0.001"/>
+        </geometry>
+        <material name="white"/>
+    </visual>
+    <inertial>
+      <origin xyz="0 0 0" rpy="0 0 0"/>
+      <mass value="1"/>
+      <inertia ixx="1.0" ixy="0.0" ixz="0.0" iyy="1.0" iyz="0.0" izz="1.0" />
+    </inertial>
+  </link>
+<!-- head_pitch -->
+  <joint name="head_pitch_joint" type="revolute">
+    <origin xyz="0 0 0" rpy="0 0 0"/>
+    <parent link="head_yaw"/>
+    <child link="head_pitch"/>
+    <axis xyz="0 1 0"/>
+    <limit velocity="6.5" effort="1000" lower="${-pi}" upper="${pi}" />
+    <dynamics damping = "0.7"/>
+  </joint>
+<transmission name="head_pitch_joint_tran">
+     <type>transmission_interface/SimpleTransmission</type>
+     <joint name="head_pitch_joint">
+       <hardwareInterface>EffortJointInterface</hardwareInterface>
+     </joint>
+     <actuator name="head_pitch_joint_motor">
+       <hardwareInterface>EffortJointInterface</hardwareInterface>
+       <mechanicalReduction>1</mechanicalReduction>
+     </actuator>
+  </transmission>
+ <link name="head_pitch">
+    <collision>
+      <origin xyz="0 0 0" rpy="0 0 0"/>
+         <geometry>
+          <mesh filename="package://erica_description/meshes/asm_don_big_main_head_pitch.stl" scale="0.001 0.001 0.001"/>
+        </geometry>
+    </collision>
+    <visual>
+        <origin xyz="0 0 0" rpy="0 0 0"/>
+        <geometry>
+          <mesh filename="package://erica_description/meshes/asm_don_big_main_head_pitch.stl" scale="0.001 0.001 0.001"/>
+        </geometry>
+        <material name="white"/>
+    </visual>
+    <inertial>
+      <origin xyz="0 0 0" rpy="0 0 0"/>
+      <mass value="1"/>
+      <inertia ixx="1.0" ixy="0.0" ixz="0.0" iyy="1.0" iyz="0.0" izz="1.0" />
+    </inertial>
+  </link>
+<!-- head_roll -->
+  <joint name="head_roll_joint" type="revolute">
+    <origin xyz="0 0 0" rpy="0 0 0"/>
+    <parent link="head_pitch"/>
+    <child link="head_roll"/>
+    <axis xyz="1 0 0"/>
+    <limit velocity="6.5" effort="1000" lower="${-pi}" upper="${pi}" />
+    <dynamics damping = "0.7"/>
+  </joint>
+<transmission name="head_roll_joint_tran">
+     <type>transmission_interface/SimpleTransmission</type>
+     <joint name="head_roll_joint">
+       <hardwareInterface>EffortJointInterface</hardwareInterface>
+     </joint>
+     <actuator name="head_roll_joint_motor">
+       <hardwareInterface>EffortJointInterface</hardwareInterface>
+       <mechanicalReduction>1</mechanicalReduction>
+     </actuator>
+  </transmission>
+ <link name="head_roll">
+    <collision>
+      <origin xyz="0 0 0" rpy="0 0 0"/>
+         <geometry>
+          <mesh filename="package://erica_description/meshes/asm_don_big_main_head_roll.stl" scale="0.001 0.001 0.001"/>
+        </geometry>
+    </collision>
+    <visual>
+        <origin xyz="0 0 0" rpy="0 0 0"/>
+        <geometry>
+          <mesh filename="package://erica_description/meshes/asm_don_big_main_head_roll.stl" scale="0.001 0.001 0.001"/>
+        </geometry>
+        <material name="white"/>
+    </visual>
+    <inertial>
+      <origin xyz="0 0 0" rpy="0 0 0"/>
+      <mass value="1"/>
       <inertia ixx="1.0" ixy="0.0" ixz="0.0" iyy="1.0" iyz="0.0" izz="1.0" />
     </inertial>
@@ -45,10 +344,29 @@
   <!-- head(zed) -->
    <joint name="camera_joint" type="fixed">
-    <parent link="body_main"/>
+    <parent link="head_roll"/>
     <child link="zed_camera_center"/>
-    <origin xyz="0.09 0 0.195" rpy="0 0 0"/>
+    <origin xyz="0.0778 0 0" rpy="0 0 0"/>
   </joint>
   <!-- Camera Center -->
-  <link name="zed_camera_center"/>
+  <link name="zed_camera_center">
+    <collision>
+      <origin xyz="0 0 0" rpy="0 0 0"/>
+      <geometry>
+          <mesh filename="package://erica_description/meshes/asm_don_big_main_zed.stl" scale="0.001 0.001 0.001"/>
+        </geometry>
+    </collision>
+    <visual>
+        <origin xyz="0 0 0" rpy="0 0 0"/>
+        <geometry>
+          <mesh filename="package://erica_description/meshes/asm_don_big_main_zed.stl" scale="0.001 0.001 0.001"/>
+        </geometry>
+        <material name="white"/>
+    </visual>
+    <inertial>
+      <origin xyz="0 0 0" rpy="0 0 0"/>
+      <mass value="1"/>
+      <inertia ixx="1.0" ixy="0.0" ixz="0.0" iyy="1.0" iyz="0.0" izz="1.0" />
+    </inertial>
+  </link>
   <!-- Left Camera -->
   <joint name="zed_left_camera_joint" type="fixed">
@@ -82,5 +400,5 @@
     <parent link="body_main"/>
     <child link="l_arm_shoulder_pitch_link"/>
-    <origin xyz="0 0.113 0" rpy="0 0 0"/>
+    <origin xyz="0 0.113 0.897" rpy="0 0 0"/>
     <axis xyz="0 1 0"/>
     <limit velocity="6.5" effort="1000" lower="${-pi}" upper="${pi}" />
@@ -317,5 +635,5 @@
     <parent link="body_main"/>
     <child link="r_arm_shoulder_pitch_link"/>
-    <origin xyz="0 -0.113 0" rpy="0 0 0"/>
+    <origin xyz="0 -0.113 0.897" rpy="0 0 0"/>
     <axis xyz="0 -1 0"/>
     <limit velocity="6.5" effort="1000" lower="${-pi}" upper="${pi}" />
