Commit message: upload working files

File: erica_description/urdf/erica_robot.xacro (robot description, xacro)
@@ -1,6 +1,6 @@
 <?xml version="1.0"?>
 <robot name="erica_robot" xmlns:xacro="http://www.ros.org/wiki/xacro">
-  <xacro:property name="pi" value="3.14" />
-   <!-- Import all Gazebo-customization elements, including Gazebo colors -->
+  <xacro:property name="pi" value="3.14159" />
+  <!-- Import all Gazebo-customization elements, including Gazebo colors -->
   <xacro:include filename="$(find erica_description)/urdf/erica_gazebo.gazebo" />
   <xacro:include filename="$(find erica_description)/urdf/materials.xacro" />
@@ -23,17 +23,17 @@
 -->
   <!-- main -->
- <link name="body_main">
-    <collision>
-      <origin xyz="0 0 0" rpy="0 0 0"/>
-         <geometry>
+  <link name="body_main">
+    <collision>
+      <origin xyz="0 0 0" rpy="0 0 0"/>
+        <geometry>
           <mesh filename="package://erica_description/meshes/asm_don_big_main.stl" scale="0.001 0.001 0.001"/>
         </geometry>
     </collision>
     <visual>
-        <origin xyz="0 0 0" rpy="0 0 0"/>
-        <geometry>
-          <mesh filename="package://erica_description/meshes/asm_don_big_main.stl" scale="0.001 0.001 0.001"/>
-        </geometry>
-        <material name="white"/>
+      <origin xyz="0 0 0" rpy="0 0 0"/>
+      <geometry>
+        <mesh filename="package://erica_description/meshes/asm_don_big_main.stl" scale="0.001 0.001 0.001"/>
+      </geometry>
+      <material name="white"/>
     </visual>
     <inertial>
@@ -52,5 +52,5 @@
     <dynamics damping = "0.7"/>
   </joint>
-<transmission name="left_wheel_front_joint_tran">
+  <transmission name="left_wheel_front_joint_tran">
      <type>transmission_interface/SimpleTransmission</type>
      <joint name="left_wheel_front_joint">
@@ -91,5 +91,5 @@
     <dynamics damping = "0.7"/>
   </joint>
-<transmission name="right_wheel_front_joint_tran">
+  <transmission name="right_wheel_front_joint_tran">
      <type>transmission_interface/SimpleTransmission</type>
      <joint name="right_wheel_front_joint">
@@ -375,5 +375,5 @@
    <origin xyz="0 0.06 0" rpy="0 0 0" />
   </joint>
-    <link name="zed_left_camera_frame" />
+  <link name="zed_left_camera_frame" />
   <joint name="zed_left_camera_optical_joint" type="fixed">
     <origin xyz="0 0 0" rpy="-1.57079632679 0.0 -1.57079632679"/>

Commit message: head gazebo added

File: erica_description/urdf/erica_robot.xacro (robot description, xacro)
@@ -203,7 +203,7 @@
     <origin xyz="0 0 0.933" rpy="0 0 0"/>
     <parent link="body_main"/>
-    <child link="neck_joint"/>
-  </joint>
- <link name="neck_joint">
+    <child link="neck_link"/>
+  </joint>
+ <link name="neck_link">
     <collision>
       <origin xyz="0 0 0" rpy="0 0 0"/>
@@ -226,23 +226,23 @@
   </link>
 <!-- head_yaw -->
-  <joint name="head_yaw_joint" type="revolute">
+  <joint name="head_yaw" type="revolute">
     <origin xyz="0 0 0.164" rpy="0 0 0"/>
-    <parent link="neck_joint"/>
-    <child link="head_yaw"/>
+    <parent link="neck_link"/>
+    <child link="head_yaw_link"/>
     <axis xyz="0 0 1"/>
     <limit velocity="6.5" effort="1000" lower="${-pi}" upper="${pi}" />
     <dynamics damping = "0.7"/>
   </joint>
-<transmission name="head_yaw_joint_tran">
-     <type>transmission_interface/SimpleTransmission</type>
-     <joint name="head_yaw_joint">
-       <hardwareInterface>EffortJointInterface</hardwareInterface>
-     </joint>
-     <actuator name="head_yaw_joint_motor">
-       <hardwareInterface>EffortJointInterface</hardwareInterface>
-       <mechanicalReduction>1</mechanicalReduction>
-     </actuator>
-  </transmission>
- <link name="head_yaw">
+<transmission name="head_yaw_tran">
+     <type>transmission_interface/SimpleTransmission</type>
+     <joint name="head_yaw">
+       <hardwareInterface>EffortJointInterface</hardwareInterface>
+     </joint>
+     <actuator name="head_yaw_motor">
+       <hardwareInterface>EffortJointInterface</hardwareInterface>
+       <mechanicalReduction>1</mechanicalReduction>
+     </actuator>
+  </transmission>
+ <link name="head_yaw_link">
     <collision>
       <origin xyz="0 0 0" rpy="0 0 0"/>
@@ -265,23 +265,23 @@
   </link>
 <!-- head_pitch -->
-  <joint name="head_pitch_joint" type="revolute">
+  <joint name="head_pitch" type="revolute">
     <origin xyz="0 0 0" rpy="0 0 0"/>
-    <parent link="head_yaw"/>
-    <child link="head_pitch"/>
-    <axis xyz="0 1 0"/>
-    <limit velocity="6.5" effort="1000" lower="${-pi}" upper="${pi}" />
-    <dynamics damping = "0.7"/>
-  </joint>
-<transmission name="head_pitch_joint_tran">
-     <type>transmission_interface/SimpleTransmission</type>
-     <joint name="head_pitch_joint">
-       <hardwareInterface>EffortJointInterface</hardwareInterface>
-     </joint>
-     <actuator name="head_pitch_joint_motor">
-       <hardwareInterface>EffortJointInterface</hardwareInterface>
-       <mechanicalReduction>1</mechanicalReduction>
-     </actuator>
-  </transmission>
- <link name="head_pitch">
+    <parent link="head_yaw_link"/>
+    <child link="head_pitch_link"/>
+    <axis xyz="0 -1 0"/>
+    <limit velocity="6.5" effort="1000" lower="${-pi}" upper="${pi}" />
+    <dynamics damping = "0.7"/>
+  </joint>
+<transmission name="head_pitch_tran">
+     <type>transmission_interface/SimpleTransmission</type>
+     <joint name="head_pitch">
+       <hardwareInterface>EffortJointInterface</hardwareInterface>
+     </joint>
+     <actuator name="head_pitch_motor">
+       <hardwareInterface>EffortJointInterface</hardwareInterface>
+       <mechanicalReduction>1</mechanicalReduction>
+     </actuator>
+  </transmission>
+ <link name="head_pitch_link">
     <collision>
       <origin xyz="0 0 0" rpy="0 0 0"/>
@@ -304,23 +304,23 @@
   </link>
 <!-- head_roll -->
-  <joint name="head_roll_joint" type="revolute">
+  <joint name="head_roll" type="revolute">
     <origin xyz="0 0 0" rpy="0 0 0"/>
-    <parent link="head_pitch"/>
-    <child link="head_roll"/>
+    <parent link="head_pitch_link"/>
+    <child link="head_roll_link"/>
     <axis xyz="1 0 0"/>
     <limit velocity="6.5" effort="1000" lower="${-pi}" upper="${pi}" />
     <dynamics damping = "0.7"/>
   </joint>
-<transmission name="head_roll_joint_tran">
-     <type>transmission_interface/SimpleTransmission</type>
-     <joint name="head_roll_joint">
-       <hardwareInterface>EffortJointInterface</hardwareInterface>
-     </joint>
-     <actuator name="head_roll_joint_motor">
-       <hardwareInterface>EffortJointInterface</hardwareInterface>
-       <mechanicalReduction>1</mechanicalReduction>
-     </actuator>
-  </transmission>
- <link name="head_roll">
+<transmission name="head_roll_tran">
+     <type>transmission_interface/SimpleTransmission</type>
+     <joint name="head_roll">
+       <hardwareInterface>EffortJointInterface</hardwareInterface>
+     </joint>
+     <actuator name="head_roll_motor">
+       <hardwareInterface>EffortJointInterface</hardwareInterface>
+       <mechanicalReduction>1</mechanicalReduction>
+     </actuator>
+  </transmission>
+ <link name="head_roll_link">
     <collision>
       <origin xyz="0 0 0" rpy="0 0 0"/>
@@ -344,5 +344,5 @@
   <!-- head(zed) -->
    <joint name="camera_joint" type="fixed">
-    <parent link="head_roll"/>
+    <parent link="head_roll_link"/>
     <child link="zed_camera_center"/>
     <origin xyz="0.0778 0 0" rpy="0 0 0"/>

Commit message: re-arrange urdf and gazebo files

File: erica_description/urdf/erica_robot.xacro (robot description, xacro)
@@ -130,5 +130,5 @@
     <dynamics damping = "0.7"/>
   </joint>
-<transmission name="left_wheel_rear_joint_tran">
+  <transmission name="left_wheel_rear_joint_tran">
      <type>transmission_interface/SimpleTransmission</type>
      <joint name="left_wheel_rear_joint">
@@ -140,5 +140,5 @@
      </actuator>
   </transmission>
- <link name="left_wheel_rear">
+  <link name="left_wheel_rear">
     <collision>
       <origin xyz="0 0 0" rpy="0 0 0"/>
@@ -160,5 +160,5 @@
     </inertial>
   </link>
- <!-- right wheel rear -->
+  <!-- right wheel rear -->
   <joint name="right_wheel_rear_joint" type="revolute">
     <origin xyz="-0.09 -0.157 0.037" rpy="0 0 0"/>
@@ -169,5 +169,5 @@
     <dynamics damping = "0.7"/>
   </joint>
-<transmission name="right_wheel_rear_joint_tran">
+  <transmission name="right_wheel_rear_joint_tran">
      <type>transmission_interface/SimpleTransmission</type>
      <joint name="right_wheel_rear_joint">
@@ -179,5 +179,5 @@
      </actuator>
   </transmission>
- <link name="right_wheel_rear">
+  <link name="right_wheel_rear">
     <collision>
       <origin xyz="0 0 0" rpy="0 0 0"/>
@@ -199,5 +199,5 @@
     </inertial>
   </link>
-<!-- neck-->
+  <!-- neck-->
   <joint name="neck_fixed_joint" type="fixed">
     <origin xyz="0 0 0.933" rpy="0 0 0"/>
@@ -205,5 +205,5 @@
     <child link="neck_link"/>
   </joint>
- <link name="neck_link">
+  <link name="neck_link">
     <collision>
       <origin xyz="0 0 0" rpy="0 0 0"/>
@@ -264,5 +264,5 @@
     </inertial>
   </link>
-<!-- head_pitch -->
+  <!-- head_pitch -->
   <joint name="head_pitch" type="revolute">
     <origin xyz="0 0 0" rpy="0 0 0"/>
@@ -273,5 +273,5 @@
     <dynamics damping = "0.7"/>
   </joint>
-<transmission name="head_pitch_tran">
+  <transmission name="head_pitch_tran">
      <type>transmission_interface/SimpleTransmission</type>
      <joint name="head_pitch">
@@ -283,5 +283,5 @@
      </actuator>
   </transmission>
- <link name="head_pitch_link">
+  <link name="head_pitch_link">
     <collision>
       <origin xyz="0 0 0" rpy="0 0 0"/>
@@ -303,5 +303,5 @@
     </inertial>
   </link>
-<!-- head_roll -->
+  <!-- head_roll -->
   <joint name="head_roll" type="revolute">
     <origin xyz="0 0 0" rpy="0 0 0"/>
@@ -312,5 +312,5 @@
     <dynamics damping = "0.7"/>
   </joint>
-<transmission name="head_roll_tran">
+  <transmission name="head_roll_tran">
      <type>transmission_interface/SimpleTransmission</type>
      <joint name="head_roll">
@@ -322,5 +322,5 @@
      </actuator>
   </transmission>
- <link name="head_roll_link">
+  <link name="head_roll_link">
     <collision>
       <origin xyz="0 0 0" rpy="0 0 0"/>
@@ -343,5 +343,5 @@
   </link>
   <!-- head(zed) -->
-   <joint name="camera_joint" type="fixed">
+  <joint name="camera_joint" type="fixed">
     <parent link="head_roll_link"/>
     <child link="zed_camera_center"/>
@@ -436,5 +436,5 @@
   </link>
   <!-- left_arm_roll -->
- <joint name="l_arm_sh_r" type="revolute">
+  <joint name="l_arm_sh_r" type="revolute">
     <parent link="l_arm_shoulder_pitch_link"/>
     <child link="l_arm_shoulder_roll_link"/>
@@ -475,5 +475,5 @@
   </link>
   <!-- left_arm_yaw -->
-<joint name="l_arm_sh_y" type="revolute">
+  <joint name="l_arm_sh_y" type="revolute">
     <parent link="l_arm_shoulder_roll_link"/>
     <child link="l_arm_shoulder_yaw_link"/>
@@ -514,5 +514,5 @@
   </link>
   <!-- left_arm_elbow -->
-<joint name="l_arm_el_p" type="revolute">
+  <joint name="l_arm_el_p" type="revolute">
     <parent link="l_arm_shoulder_yaw_link"/>
     <child link="l_arm_elbow_pitch_link"/>
@@ -553,5 +553,5 @@
   </link>
   <!-- left_arm_wrist_pitch -->
-<joint name="l_arm_wr_p" type="revolute">
+  <joint name="l_arm_wr_p" type="revolute">
     <parent link="l_arm_elbow_pitch_link"/>
     <child link="l_arm_wrist_pitch_link"/>
@@ -591,6 +591,6 @@
     </inertial>
   </link>
-<!-- left_arm_wrist_roll -->
-<joint name="l_arm_wr_r" type="revolute">
+  <!-- left_arm_wrist_roll -->
+  <joint name="l_arm_wr_r" type="revolute">
     <parent link="l_arm_wrist_pitch_link"/>
     <child link="l_arm_wrist_roll_link"/>
@@ -630,7 +630,7 @@
     </inertial>
   </link>
-    <!-- right_arm -->
+  <!-- right_arm -->
   <!-- right_arm_pitch -->
- <joint name="r_arm_sh_p" type="revolute">
+  <joint name="r_arm_sh_p" type="revolute">
     <parent link="body_main"/>
     <child link="r_arm_shoulder_pitch_link"/>
@@ -671,5 +671,5 @@
   </link>
   <!-- right_arm_roll -->
- <joint name="r_arm_sh_r" type="revolute">
+  <joint name="r_arm_sh_r" type="revolute">
     <parent link="r_arm_shoulder_pitch_link"/>
     <child link="r_arm_shoulder_roll_link"/>
@@ -710,5 +710,5 @@
   </link>
   <!-- right_arm_yaw -->
-<joint name="r_arm_sh_y" type="revolute">
+  <joint name="r_arm_sh_y" type="revolute">
     <parent link="r_arm_shoulder_roll_link"/>
     <child link="r_arm_shoulder_yaw_link"/>
@@ -749,5 +749,5 @@
   </link>
   <!-- right_arm_elbow -->
-<joint name="r_arm_el_p" type="revolute">
+  <joint name="r_arm_el_p" type="revolute">
     <parent link="r_arm_shoulder_yaw_link"/>
     <child link="r_arm_elbow_pitch_link"/>
@@ -788,5 +788,5 @@
   </link>
   <!-- right_arm_wrist_pitch -->
-<joint name="r_arm_wr_p" type="revolute">
+  <joint name="r_arm_wr_p" type="revolute">
     <parent link="r_arm_elbow_pitch_link"/>
     <child link="r_arm_wrist_pitch_link"/>
@@ -827,5 +827,5 @@
   </link>
 <!-- right_arm_wrist_roll -->
-<joint name="r_arm_wr_r" type="revolute">
+  <joint name="r_arm_wr_r" type="revolute">
     <parent link="r_arm_wrist_pitch_link"/>
     <child link="r_arm_wrist_roll_link"/>
