Commit message: omni wheel dummy completed

File: erica_description/urdf/erica_robot.xacro (robot description, xacro)
@@ -39,17 +39,57 @@
     <inertial>
       <origin xyz="0 0 0" rpy="0 0 0"/>
-      <mass value="300"/>
-      <inertia ixx="1.0" ixy="0.0" ixz="0.0" iyy="1.0" iyz="0.0" izz="1.0" />
-    </inertial>
-  </link>
-  <!-- left wheel front-->
-  <joint name="left_wheel_front_joint" type="revolute">
+      <mass value="50"/>
+      <inertia ixx="1.0" ixy="0.0" ixz="0.0" iyy="1.0" iyz="0.0" izz="1.0" />
+    </inertial>
+  </link>
+  <!-- left wheel front steering-->
+  <joint name="left_wheel_front_steering_joint" type="revolute">
     <origin xyz="0.09 0.157 0.037" rpy="0 0 0"/>
     <parent link="body_main"/>
+    <child link="left_wheel_front_steering"/>
+    <axis xyz="0 0 1"/>
+    <limit velocity="6.5" effort="1000" lower="${-pi}" upper="${pi}" />
+    <dynamics damping = "0.7"/>
+  </joint>
+  <transmission name="left_wheel_front_steering_joint_tran">
+     <type>transmission_interface/SimpleTransmission</type>
+     <joint name="left_wheel_front_steering_joint">
+       <hardwareInterface>EffortJointInterface</hardwareInterface>
+     </joint>
+     <actuator name="left_wheel_front_steering_joint_motor">
+       <hardwareInterface>EffortJointInterface</hardwareInterface>
+       <mechanicalReduction>1</mechanicalReduction>
+     </actuator>
+  </transmission>
+  <link name="left_wheel_front_steering">
+    <collision>
+      <origin xyz="0 0 0" rpy="0 0 0"/>
+         <geometry>
+           <box size="0.001 0.001 0.001" />
+        </geometry>
+    </collision>
+    <visual>
+        <origin xyz="0 0 0" rpy="0 0 0"/>
+        <geometry>
+          <box size="0.001 0.001 0.001" />
+        </geometry>
+        <material name="white"/>
+    </visual>
+    <inertial>
+      <origin xyz="0 0 0" rpy="0 0 0"/>
+      <mass value="2.5"/>
+      <inertia ixx="1.0" ixy="0.0" ixz="0.0" iyy="1.0" iyz="0.0" izz="1.0" />
+    </inertial>
+  </link>
+  <!-- left wheel front-->
+  <joint name="left_wheel_front_joint" type="continuous">
+    <origin xyz="0 0 0" rpy="0 0 0"/>
+    <parent link="left_wheel_front_steering"/>
     <child link="left_wheel_front"/>
     <axis xyz="0 1 0"/>
-    <limit velocity="6.5" effort="1000" lower="${-pi}" upper="${pi}" />
-    <dynamics damping = "0.7"/>
-  </joint>
+  <!-- <limit velocity="6.5" effort="1000" lower="${-pi}" upper="${pi}" />-->
+    <dynamics damping = "0.7"/>
+  </joint>
+ <!--
   <transmission name="left_wheel_front_joint_tran">
      <type>transmission_interface/SimpleTransmission</type>
@@ -62,4 +102,5 @@
      </actuator>
   </transmission>
+-->
  <link name="left_wheel_front">
     <collision>
@@ -68,4 +109,12 @@
           <mesh filename="package://erica_description/meshes/left_wheel_front.stl" scale="0.001 0.001 0.001"/>
         </geometry>
+        <surface>
+          <friction>
+            <ode>
+              <mu>0.001</mu>
+              <mu2>0.001</mu2>
+            </ode>
+          </friction>
+        </surface>
     </collision>
     <visual>
@@ -78,17 +127,57 @@
     <inertial>
       <origin xyz="0 0 0" rpy="0 0 0"/>
-      <mass value="1"/>
-      <inertia ixx="1.0" ixy="0.0" ixz="0.0" iyy="1.0" iyz="0.0" izz="1.0" />
-    </inertial>
-  </link>
- <!-- right wheel front -->
-  <joint name="right_wheel_front_joint" type="revolute">
+      <mass value="2.5"/>
+      <inertia ixx="1.0" ixy="0.0" ixz="0.0" iyy="1.0" iyz="0.0" izz="1.0" />
+    </inertial>
+  </link>
+    <!-- right wheel front steering-->
+  <joint name="right_wheel_front_steering_joint" type="revolute">
     <origin xyz="0.09 -0.157 0.037" rpy="0 0 0"/>
     <parent link="body_main"/>
+    <child link="right_wheel_front_steering"/>
+    <axis xyz="0 0 1"/>
+    <limit velocity="6.5" effort="1000" lower="${-pi}" upper="${pi}" />
+    <dynamics damping = "0.7"/>
+  </joint>
+  <transmission name="right_wheel_front_steering_joint_tran">
+     <type>transmission_interface/SimpleTransmission</type>
+     <joint name="right_wheel_front_steering_joint">
+       <hardwareInterface>EffortJointInterface</hardwareInterface>
+     </joint>
+     <actuator name="right_wheel_front_steering_joint_motor">
+       <hardwareInterface>EffortJointInterface</hardwareInterface>
+       <mechanicalReduction>1</mechanicalReduction>
+     </actuator>
+  </transmission>
+ <link name="right_wheel_front_steering">
+    <collision>
+      <origin xyz="0 0 0" rpy="0 0 0"/>
+         <geometry>
+           <box size="0.001 0.001 0.001" />
+        </geometry>
+    </collision>
+    <visual>
+        <origin xyz="0 0 0" rpy="0 0 0"/>
+        <geometry>
+          <box size="0.001 0.001 0.001" />
+        </geometry>
+        <material name="white"/>
+    </visual>
+    <inertial>
+      <origin xyz="0 0 0" rpy="0 0 0"/>
+      <mass value="2.5"/>
+      <inertia ixx="1.0" ixy="0.0" ixz="0.0" iyy="1.0" iyz="0.0" izz="1.0" />
+    </inertial>
+  </link>
+ <!-- right wheel front -->
+  <joint name="right_wheel_front_joint" type="continuous">
+    <origin xyz="0 0 0" rpy="0 0 0"/>
+    <parent link="right_wheel_front_steering"/>
     <child link="right_wheel_front"/>
     <axis xyz="0 1 0"/>
-    <limit velocity="6.5" effort="1000" lower="${-pi}" upper="${pi}" />
-    <dynamics damping = "0.7"/>
-  </joint>
+ <!--<limit velocity="6.5" effort="1000" lower="${-pi}" upper="${pi}" />-->
+    <dynamics damping = "0.7"/>
+  </joint>
+ <!--
   <transmission name="right_wheel_front_joint_tran">
      <type>transmission_interface/SimpleTransmission</type>
@@ -101,4 +190,5 @@
      </actuator>
   </transmission>
+-->
  <link name="right_wheel_front">
     <collision>
@@ -107,4 +197,12 @@
           <mesh filename="package://erica_description/meshes/right_wheel_front.stl" scale="0.001 0.001 0.001"/>
         </geometry>
+        <surface>
+          <friction>
+            <ode>
+              <mu>0.001</mu>
+              <mu2>0.001</mu2>
+            </ode>
+          </friction>
+        </surface>
     </collision>
     <visual>
@@ -121,13 +219,53 @@
     </inertial>
   </link>
-  <!-- left wheel rear-->
-  <joint name="left_wheel_rear_joint" type="revolute">
+  <!-- left wheel rear steering-->
+  <joint name="left_wheel_rear_steering_joint" type="revolute">
     <origin xyz="-0.09 0.157 0.037" rpy="0 0 0"/>
     <parent link="body_main"/>
+    <child link="left_wheel_rear_steering"/>
+    <axis xyz="0 0 1"/>
+    <limit velocity="6.5" effort="1000" lower="${-pi}" upper="${pi}" />
+    <dynamics damping = "0.7"/>
+  </joint>
+  <transmission name="left_wheel_rear_steering_joint_tran">
+     <type>transmission_interface/SimpleTransmission</type>
+     <joint name="left_wheel_rear_steering_joint">
+       <hardwareInterface>EffortJointInterface</hardwareInterface>
+     </joint>
+     <actuator name="left_wheel_rear_steering_joint_motor">
+       <hardwareInterface>EffortJointInterface</hardwareInterface>
+       <mechanicalReduction>1</mechanicalReduction>
+     </actuator>
+  </transmission>
+  <link name="left_wheel_rear_steering">
+    <collision>
+      <origin xyz="0 0 0" rpy="0 0 0"/>
+         <geometry>
+           <box size="0.001 0.001 0.001" />
+        </geometry>
+    </collision>
+    <visual>
+        <origin xyz="0 0 0" rpy="0 0 0"/>
+        <geometry>
+          <box size="0.001 0.001 0.001" />
+        </geometry>
+        <material name="white"/>
+    </visual>
+    <inertial>
+      <origin xyz="0 0 0" rpy="0 0 0"/>
+      <mass value="2.5"/>
+      <inertia ixx="1.0" ixy="0.0" ixz="0.0" iyy="1.0" iyz="0.0" izz="1.0" />
+    </inertial>
+  </link>
+  <!-- left wheel rear-->
+  <joint name="left_wheel_rear_joint" type="continuous">
+    <origin xyz="0 0 0" rpy="0 0 0"/>
+    <parent link="left_wheel_rear_steering"/>
     <child link="left_wheel_rear"/>
     <axis xyz="0 1 0"/>
-    <limit velocity="6.5" effort="1000" lower="${-pi}" upper="${pi}" />
-    <dynamics damping = "0.7"/>
-  </joint>
+   <!--<limit velocity="6.5" effort="1000" lower="${-pi}" upper="${pi}" /> -->
+    <dynamics damping = "0.7"/>
+  </joint>
+<!--
   <transmission name="left_wheel_rear_joint_tran">
      <type>transmission_interface/SimpleTransmission</type>
@@ -140,4 +278,5 @@
      </actuator>
   </transmission>
+-->
   <link name="left_wheel_rear">
     <collision>
@@ -146,4 +285,12 @@
           <mesh filename="package://erica_description/meshes/left_wheel_rear.stl" scale="0.001 0.001 0.001"/>
         </geometry>
+        <surface>
+          <friction>
+            <ode>
+              <mu>0.001</mu>
+              <mu2>0.001</mu2>
+            </ode>
+          </friction>
+        </surface>
     </collision>
     <visual>
@@ -156,17 +303,57 @@
     <inertial>
       <origin xyz="0 0 0" rpy="0 0 0"/>
-      <mass value="1"/>
-      <inertia ixx="1.0" ixy="0.0" ixz="0.0" iyy="1.0" iyz="0.0" izz="1.0" />
-    </inertial>
-  </link>
-  <!-- right wheel rear -->
-  <joint name="right_wheel_rear_joint" type="revolute">
+      <mass value="2.5"/>
+      <inertia ixx="1.0" ixy="0.0" ixz="0.0" iyy="1.0" iyz="0.0" izz="1.0" />
+    </inertial>
+  </link>
+  <!-- right wheel rear steering-->
+  <joint name="right_wheel_rear_steering_joint" type="revolute">
     <origin xyz="-0.09 -0.157 0.037" rpy="0 0 0"/>
     <parent link="body_main"/>
+    <child link="right_wheel_rear_steering"/>
+    <axis xyz="0 0 1"/>
+    <limit velocity="6.5" effort="1000" lower="${-pi}" upper="${pi}" />
+    <dynamics damping = "0.7"/>
+  </joint>
+  <transmission name="right_wheel_rear_steering_joint_tran">
+     <type>transmission_interface/SimpleTransmission</type>
+     <joint name="right_wheel_rear_steering_joint">
+       <hardwareInterface>EffortJointInterface</hardwareInterface>
+     </joint>
+     <actuator name="right_wheel_rear_steering_joint_motor">
+       <hardwareInterface>EffortJointInterface</hardwareInterface>
+       <mechanicalReduction>1</mechanicalReduction>
+     </actuator>
+  </transmission>
+  <link name="right_wheel_rear_steering">
+    <collision>
+      <origin xyz="0 0 0" rpy="0 0 0"/>
+         <geometry>
+           <box size="0.001 0.001 0.001" />
+        </geometry>
+    </collision>
+    <visual>
+        <origin xyz="0 0 0" rpy="0 0 0"/>
+        <geometry>
+          <box size="0.001 0.001 0.001" />
+        </geometry>
+        <material name="white"/>
+    </visual>
+    <inertial>
+      <origin xyz="0 0 0" rpy="0 0 0"/>
+      <mass value="2.5"/>
+      <inertia ixx="1.0" ixy="0.0" ixz="0.0" iyy="1.0" iyz="0.0" izz="1.0" />
+    </inertial>
+  </link>
+  <!-- right wheel rear -->
+  <joint name="right_wheel_rear_joint" type="continuous">
+    <origin xyz="0 0 0" rpy="0 0 0"/>
+    <parent link="right_wheel_rear_steering"/>
     <child link="right_wheel_rear"/>
     <axis xyz="0 1 0"/>
-    <limit velocity="6.5" effort="1000" lower="${-pi}" upper="${pi}" />
-    <dynamics damping = "0.7"/>
-  </joint>
+  <!--<limit velocity="6.5" effort="1000" lower="${-pi}" upper="${pi}" />-->
+    <dynamics damping = "0.7"/>
+  </joint>
+<!--
   <transmission name="right_wheel_rear_joint_tran">
      <type>transmission_interface/SimpleTransmission</type>
@@ -179,4 +366,5 @@
      </actuator>
   </transmission>
+-->
   <link name="right_wheel_rear">
     <collision>
@@ -185,4 +373,12 @@
           <mesh filename="package://erica_description/meshes/right_wheel_rear.stl" scale="0.001 0.001 0.001"/>
         </geometry>
+        <surface>
+          <friction>
+            <ode>
+              <mu>0.001</mu>
+              <mu2>0.001</mu2>
+            </ode>
+          </friction>
+        </surface>
     </collision>
     <visual>

Commit message: model modified

File: erica_description/urdf/erica_robot.xacro (robot description, xacro)
@@ -6,27 +6,11 @@
   <xacro:include filename="$(find erica_description)/urdf/materials.xacro" />
   <!-- Used for fixing robot -->
-<!--
-  <link name="world">
-  </link>
-  <joint name="world_fixed" type="fixed">
-    <origin xyz="0 0 0.7" rpy="0 0 0"/>
-    <parent link="world"/>
-    <child link="pelvis"/>
-  </joint>
-  <link name="base">
-  </link>
-  <joint name="base_fixed" type="fixed">
-    <origin xyz="0 0 0.2" rpy="0 0 0"/>
-    <parent link="base"/>
-    <child link="body_main"/>
-  </joint>
--->
   <!-- main -->
   <link name="body_main">
     <collision>
       <origin xyz="0 0 0" rpy="0 0 0"/>
-        <geometry>
-          <mesh filename="package://erica_description/meshes/asm_don_big_main.stl" scale="0.001 0.001 0.001"/>
-        </geometry>
+      <geometry>
+        <mesh filename="package://erica_description/meshes/asm_don_big_main.stl" scale="0.001 0.001 0.001"/>
+      </geometry>
     </collision>
     <visual>
@@ -41,4 +25,30 @@
       <mass value="50"/>
       <inertia ixx="1.0" ixy="0.0" ixz="0.0" iyy="1.0" iyz="0.0" izz="1.0" />
+    </inertial>
+  </link>
+  <joint name="hokuyo_joint" type="fixed">
+    <axis xyz="0 1 0" />
+    <origin xyz="0.05 0 0.25" rpy="0 0 0"/>
+    <parent link="body_main"/>
+    <child link="hokuyo_link"/>
+  </joint>
+    <!-- Hokuyo Laser -->
+  <link name="hokuyo_link">
+    <collision>
+      <origin xyz="0 0 0" rpy="0 0 0"/>
+      <geometry>
+        <box size="0.05 0.05 0.05"/>
+      </geometry>
+    </collision>
+    <visual>
+      <origin xyz="0 0 0" rpy="0 0 0"/>
+      <geometry>
+        <box size="0.05 0.05 0.05"/>
+      </geometry>
+    </visual>
+    <inertial>
+      <mass value="1e-5" />
+      <origin xyz="0 0 0" rpy="0 0 0"/>
+      <inertia ixx="1e-6" ixy="0" ixz="0" iyy="1e-6" iyz="0" izz="1e-6" />
     </inertial>
   </link>

Commit message: model modified

File: erica_description/urdf/erica_robot.xacro (robot description, xacro)
@@ -7,4 +7,103 @@
   <!-- Used for fixing robot -->
   <!-- main -->
+  <link name="world">
+  </link>
+  <joint name="fake_x_joint" type="prismatic">
+    <origin xyz="0 0 0" rpy="0 0 0"/>
+    <parent link="world"/>
+    <child link="fake_x_link"/>
+    <axis xyz="1 0 0"/>
+    <limit effort="6.5" lower="-1000" upper="1000" velocity="50.0" />
+  </joint>
+  <transmission name="fake_x_joint_tran">
+    <type>transmission_interface/SimpleTransmission</type>
+    <joint name="fake_x_joint">
+      <hardwareInterface>EffortJointInterface</hardwareInterface>
+    </joint>
+    <actuator name="fake_x_joint_motor">
+      <hardwareInterface>EffortJointInterface</hardwareInterface>
+      <mechanicalReduction>1</mechanicalReduction>
+    </actuator>
+  </transmission>
+  <link name="fake_x_link">
+    <visual>
+      <origin xyz="0 0 0" rpy="0 0 0"/>
+      <geometry>
+        <box size="0.005 0.005 0.005"/>
+      </geometry>
+    </visual>
+    <inertial>
+      <origin xyz="0 0 0" rpy="0 0 0"/>
+      <mass value="0.05"/>
+      <inertia ixx="1.0" ixy="0.0" ixz="0.0" iyy="1.0" iyz="0.0" izz="1.0" />
+    </inertial>
+  </link>
+  <joint name="fake_y_joint" type="prismatic">
+    <origin xyz="0 0 0" rpy="0 0 0"/>
+    <parent link="fake_x_link"/>
+    <child link="fake_y_link"/>
+    <axis xyz="0 1 0"/>
+    <limit effort="6.5" lower="-1000" upper="1000" velocity="50.0" />
+  </joint>
+  <transmission name="fake_y_joint_tran">
+    <type>transmission_interface/SimpleTransmission</type>
+    <joint name="fake_y_joint">
+      <hardwareInterface>EffortJointInterface</hardwareInterface>
+    </joint>
+    <actuator name="fake_y_joint_motor">
+      <hardwareInterface>EffortJointInterface</hardwareInterface>
+      <mechanicalReduction>1</mechanicalReduction>
+    </actuator>
+  </transmission>
+  <link name="fake_y_link">
+    <visual>
+      <origin xyz="0 0 0" rpy="0 0 0"/>
+      <geometry>
+        <box size="0.005 0.005 0.005"/>
+      </geometry>
+    </visual>
+    <inertial>
+      <origin xyz="0 0 0" rpy="0 0 0"/>
+      <mass value="0.05"/>
+      <inertia ixx="1.0" ixy="0.0" ixz="0.0" iyy="1.0" iyz="0.0" izz="1.0" />
+    </inertial>
+  </link>
+  <joint name="fake_z_joint" type="revolute">
+    <origin xyz="0 0 0" rpy="0 0 0"/>
+    <parent link="fake_y_link"/>
+    <child link="fake_z_link"/>
+    <axis xyz="0 0 1"/>
+    <limit velocity="6.5" effort="1000" lower="${-pi}" upper="${pi}" />
+    <dynamics damping = "0.7"/>
+  </joint>
+  <transmission name="fake_z_joint_tran">
+    <type>transmission_interface/SimpleTransmission</type>
+    <joint name="fake_z_joint">
+      <hardwareInterface>EffortJointInterface</hardwareInterface>
+    </joint>
+    <actuator name="fake_z_joint_motor">
+      <hardwareInterface>EffortJointInterface</hardwareInterface>
+      <mechanicalReduction>1</mechanicalReduction>
+    </actuator>
+  </transmission>
+  <link name="fake_z_link">
+    <visual>
+      <origin xyz="0 0 0" rpy="0 0 0"/>
+      <geometry>
+        <box size="0.005 0.005 0.005"/>
+      </geometry>
+    </visual>
+    <inertial>
+      <origin xyz="0 0 0" rpy="0 0 0"/>
+      <mass value="0.05"/>
+      <inertia ixx="1.0" ixy="0.0" ixz="0.0" iyy="1.0" iyz="0.0" izz="1.0" />
+    </inertial>
+  </link>
+  <joint name="fake_z_fixed_joint" type="fixed">
+    <axis xyz="0 1 0" />
+    <origin xyz="0 0 0" rpy="0 0 0"/>
+    <parent link="fake_z_link"/>
+    <child link="body_main"/>
+  </joint>
   <link name="body_main">
     <collision>
@@ -122,6 +221,6 @@
           <friction>
             <ode>
-              <mu>0.001</mu>
-              <mu2>0.001</mu2>
+              <mu>0.1</mu>
+              <mu2>1</mu2>
             </ode>
           </friction>
@@ -210,6 +309,6 @@
           <friction>
             <ode>
-              <mu>0.001</mu>
-              <mu2>0.001</mu2>
+              <mu>0.1</mu>
+              <mu2>1</mu2>
             </ode>
           </friction>
@@ -298,6 +397,6 @@
           <friction>
             <ode>
-              <mu>0.001</mu>
-              <mu2>0.001</mu2>
+              <mu>0.1</mu>
+              <mu2>1</mu2>
             </ode>
           </friction>
@@ -386,6 +485,6 @@
           <friction>
             <ode>
-              <mu>0.001</mu>
-              <mu2>0.001</mu2>
+              <mu>0.1</mu>
+              <mu2>1</mu2>
             </ode>
           </friction>
