Commit message: completed

File: erica_description/urdf/erica_robot.xacro (robot description, xacro)
@@ -5,105 +5,13 @@
   <xacro:include filename="$(find erica_description)/urdf/erica_gazebo.gazebo" />
   <xacro:include filename="$(find erica_description)/urdf/materials.xacro" />
+  <xacro:property name="base_width" value="0.26" />   <!-- 14.5 in -->
+  <xacro:property name="base_length" value="0.312" />  <!-- 21 5/8 in -->
+  <xacro:property name="base_height" value="0.105" />   <!-- 2.5 in  -->
+  <xacro:property name="wheel_radius" value="0.1016" /> <!-- 4.0 in  -->
+  <xacro:property name="wheel_width" value="0.0762" />  <!-- 3.0 in  -->
+  <xacro:property name="wheel_gap" value="0.0508" />    <!-- 2.0 in  -->
+  <xacro:property name="wheel_setback" value="0.041275" />    <!-- 1 5/8 in  -->
   <!-- Used for fixing robot -->
   <!-- main -->
-  <link name="world">
-  </link>
-  <joint name="fake_x_joint" type="prismatic">
-    <origin xyz="0 0 0" rpy="0 0 0"/>
-    <parent link="world"/>
-    <child link="fake_x_link"/>
-    <axis xyz="1 0 0"/>
-    <limit effort="6.5" lower="-1000" upper="1000" velocity="50.0" />
-  </joint>
-  <transmission name="fake_x_joint_tran">
-    <type>transmission_interface/SimpleTransmission</type>
-    <joint name="fake_x_joint">
-      <hardwareInterface>EffortJointInterface</hardwareInterface>
-    </joint>
-    <actuator name="fake_x_joint_motor">
-      <hardwareInterface>EffortJointInterface</hardwareInterface>
-      <mechanicalReduction>1</mechanicalReduction>
-    </actuator>
-  </transmission>
-  <link name="fake_x_link">
-    <visual>
-      <origin xyz="0 0 0" rpy="0 0 0"/>
-      <geometry>
-        <box size="0.005 0.005 0.005"/>
-      </geometry>
-    </visual>
-    <inertial>
-      <origin xyz="0 0 0" rpy="0 0 0"/>
-      <mass value="0.05"/>
-      <inertia ixx="1.0" ixy="0.0" ixz="0.0" iyy="1.0" iyz="0.0" izz="1.0" />
-    </inertial>
-  </link>
-  <joint name="fake_y_joint" type="prismatic">
-    <origin xyz="0 0 0" rpy="0 0 0"/>
-    <parent link="fake_x_link"/>
-    <child link="fake_y_link"/>
-    <axis xyz="0 1 0"/>
-    <limit effort="6.5" lower="-1000" upper="1000" velocity="50.0" />
-  </joint>
-  <transmission name="fake_y_joint_tran">
-    <type>transmission_interface/SimpleTransmission</type>
-    <joint name="fake_y_joint">
-      <hardwareInterface>EffortJointInterface</hardwareInterface>
-    </joint>
-    <actuator name="fake_y_joint_motor">
-      <hardwareInterface>EffortJointInterface</hardwareInterface>
-      <mechanicalReduction>1</mechanicalReduction>
-    </actuator>
-  </transmission>
-  <link name="fake_y_link">
-    <visual>
-      <origin xyz="0 0 0" rpy="0 0 0"/>
-      <geometry>
-        <box size="0.005 0.005 0.005"/>
-      </geometry>
-    </visual>
-    <inertial>
-      <origin xyz="0 0 0" rpy="0 0 0"/>
-      <mass value="0.05"/>
-      <inertia ixx="1.0" ixy="0.0" ixz="0.0" iyy="1.0" iyz="0.0" izz="1.0" />
-    </inertial>
-  </link>
-  <joint name="fake_z_joint" type="revolute">
-    <origin xyz="0 0 0" rpy="0 0 0"/>
-    <parent link="fake_y_link"/>
-    <child link="fake_z_link"/>
-    <axis xyz="0 0 1"/>
-    <limit velocity="6.5" effort="1000" lower="${-pi}" upper="${pi}" />
-    <dynamics damping = "0.7"/>
-  </joint>
-  <transmission name="fake_z_joint_tran">
-    <type>transmission_interface/SimpleTransmission</type>
-    <joint name="fake_z_joint">
-      <hardwareInterface>EffortJointInterface</hardwareInterface>
-    </joint>
-    <actuator name="fake_z_joint_motor">
-      <hardwareInterface>EffortJointInterface</hardwareInterface>
-      <mechanicalReduction>1</mechanicalReduction>
-    </actuator>
-  </transmission>
-  <link name="fake_z_link">
-    <visual>
-      <origin xyz="0 0 0" rpy="0 0 0"/>
-      <geometry>
-        <box size="0.005 0.005 0.005"/>
-      </geometry>
-    </visual>
-    <inertial>
-      <origin xyz="0 0 0" rpy="0 0 0"/>
-      <mass value="0.05"/>
-      <inertia ixx="1.0" ixy="0.0" ixz="0.0" iyy="1.0" iyz="0.0" izz="1.0" />
-    </inertial>
-  </link>
-  <joint name="fake_z_fixed_joint" type="fixed">
-    <axis xyz="0 1 0" />
-    <origin xyz="0 0 0" rpy="0 0 0"/>
-    <parent link="fake_z_link"/>
-    <child link="body_main"/>
-  </joint>
   <link name="body_main">
     <collision>
@@ -152,356 +60,108 @@
     </inertial>
   </link>
-  <!-- left wheel front steering-->
-  <joint name="left_wheel_front_steering_joint" type="revolute">
-    <origin xyz="0.09 0.157 0.037" rpy="0 0 0"/>
+  <link name="fl_link">
+    <visual>
+      <geometry>
+        <cylinder length="${wheel_width}" radius="${wheel_radius}"/>
+      </geometry>
+      <origin rpy="${pi/2} 0 0" xyz="0 0 0"/>
+    </visual>
+    <collision>
+      <geometry>
+        <cylinder length="${wheel_width}" radius="${wheel_radius}"/>
+      </geometry>
+      <origin rpy="${pi/2} 0 0" xyz="0 0 0"/>
+    </collision>
+    <inertial>
+      <mass value="2" />
+      <origin rpy="${pi/2} 0 0" xyz="0 0 0"/>
+      <inertia ixx="1e-6" ixy="0" ixz="0" iyy="1e-6" iyz="0" izz="1e-6" />
+    </inertial>
+  </link>
+  <link name="fr_link">
+    <visual>
+      <geometry>
+        <cylinder length="${wheel_width}" radius="${wheel_radius}"/>
+      </geometry>
+      <origin rpy="${pi/2} 0 0" xyz="0 0 0"/>
+    </visual>
+    <collision>
+      <geometry>
+        <cylinder length="${wheel_width}" radius="${wheel_radius}"/>
+      </geometry>
+      <origin rpy="${pi/2} 0 0" xyz="0 0 0"/>
+    </collision>
+    <inertial>
+      <mass value="2" />
+      <origin rpy="${pi/2} 0 0" xyz="0 0 0"/>
+      <inertia ixx="1e-6" ixy="0" ixz="0" iyy="1e-6" iyz="0" izz="1e-6" />
+    </inertial>
+  </link>
+  <link name="bl_link">
+    <visual>
+      <geometry>
+        <cylinder length="${wheel_width}" radius="${wheel_radius}"/>
+      </geometry>
+      <origin rpy="${pi/2} 0 0" xyz="0 0 0"/>
+    </visual>
+    <collision>
+      <geometry>
+        <cylinder length="${wheel_width}" radius="${wheel_radius}"/>
+      </geometry>
+      <origin rpy="${pi/2} 0 0" xyz="0 0 0"/>
+    </collision>
+    <inertial>
+      <mass value="2" />
+      <origin rpy="${pi/2} 0 0" xyz="0 0 0"/>
+      <inertia ixx="1e-6" ixy="0" ixz="0" iyy="1e-6" iyz="0" izz="1e-6" />
+    </inertial>
+  </link>
+  <link name="br_link">
+    <visual>
+      <geometry>
+        <cylinder length="${wheel_width}" radius="${wheel_radius}"/>
+      </geometry>
+      <origin rpy="${pi/2} 0 0" xyz="0 0 0"/>
+    </visual>
+    <collision>
+      <geometry>
+        <cylinder length="${wheel_width}" radius="${wheel_radius}"/>
+      </geometry>
+      <origin rpy="${pi/2} 0 0" xyz="0 0 0"/>
+    </collision>
+    <inertial>
+      <mass value="2" />
+      <origin rpy="${pi/2} 0 0" xyz="0 0 0"/>
+      <inertia ixx="1e-6" ixy="0" ixz="0" iyy="1e-6" iyz="0" izz="1e-6" />
+    </inertial>
+  </link>
+  <joint name="fl_joint" type="fixed">
     <parent link="body_main"/>
-    <child link="left_wheel_front_steering"/>
-    <axis xyz="0 0 1"/>
-    <limit velocity="6.5" effort="1000" lower="${-pi}" upper="${pi}" />
-    <dynamics damping = "0.7"/>
-  </joint>
-  <transmission name="left_wheel_front_steering_joint_tran">
-     <type>transmission_interface/SimpleTransmission</type>
-     <joint name="left_wheel_front_steering_joint">
-       <hardwareInterface>EffortJointInterface</hardwareInterface>
-     </joint>
-     <actuator name="left_wheel_front_steering_joint_motor">
-       <hardwareInterface>EffortJointInterface</hardwareInterface>
-       <mechanicalReduction>1</mechanicalReduction>
-     </actuator>
-  </transmission>
-  <link name="left_wheel_front_steering">
-    <collision>
-      <origin xyz="0 0 0" rpy="0 0 0"/>
-         <geometry>
-           <box size="0.001 0.001 0.001" />
-        </geometry>
-    </collision>
-    <visual>
-        <origin xyz="0 0 0" rpy="0 0 0"/>
-        <geometry>
-          <box size="0.001 0.001 0.001" />
-        </geometry>
-        <material name="white"/>
-    </visual>
-    <inertial>
-      <origin xyz="0 0 0" rpy="0 0 0"/>
-      <mass value="2.5"/>
-      <inertia ixx="1.0" ixy="0.0" ixz="0.0" iyy="1.0" iyz="0.0" izz="1.0" />
-    </inertial>
-  </link>
-  <!-- left wheel front-->
-  <joint name="left_wheel_front_joint" type="continuous">
-    <origin xyz="0 0 0" rpy="0 0 0"/>
-    <parent link="left_wheel_front_steering"/>
-    <child link="left_wheel_front"/>
-    <axis xyz="0 1 0"/>
-  <!-- <limit velocity="6.5" effort="1000" lower="${-pi}" upper="${pi}" />-->
-    <dynamics damping = "0.7"/>
-  </joint>
- <!--
-  <transmission name="left_wheel_front_joint_tran">
-     <type>transmission_interface/SimpleTransmission</type>
-     <joint name="left_wheel_front_joint">
-       <hardwareInterface>EffortJointInterface</hardwareInterface>
-     </joint>
-     <actuator name="left_wheel_front_joint_motor">
-       <hardwareInterface>EffortJointInterface</hardwareInterface>
-       <mechanicalReduction>1</mechanicalReduction>
-     </actuator>
-  </transmission>
--->
- <link name="left_wheel_front">
-    <collision>
-      <origin xyz="0 0 0" rpy="0 0 0"/>
-         <geometry>
-          <mesh filename="package://erica_description/meshes/left_wheel_front.stl" scale="0.001 0.001 0.001"/>
-        </geometry>
-        <surface>
-          <friction>
-            <ode>
-              <mu>0.1</mu>
-              <mu2>1</mu2>
-            </ode>
-          </friction>
-        </surface>
-    </collision>
-    <visual>
-        <origin xyz="0 0 0" rpy="0 0 0"/>
-        <geometry>
-          <mesh filename="package://erica_description/meshes/left_wheel_front.stl" scale="0.001 0.001 0.001"/>
-        </geometry>
-        <material name="white"/>
-    </visual>
-    <inertial>
-      <origin xyz="0 0 0" rpy="0 0 0"/>
-      <mass value="2.5"/>
-      <inertia ixx="1.0" ixy="0.0" ixz="0.0" iyy="1.0" iyz="0.0" izz="1.0" />
-    </inertial>
-  </link>
-    <!-- right wheel front steering-->
-  <joint name="right_wheel_front_steering_joint" type="revolute">
-    <origin xyz="0.09 -0.157 0.037" rpy="0 0 0"/>
+    <child link="fl_link"/>
+    <origin rpy="0 0 0" xyz="${base_length/2 - wheel_setback} ${base_width/2 + wheel_gap} 0.0"/>
+    <axis xyz="0 0 0"/>
+    <!-- <dynamics damping="1.0" friction="0.0" spring_stiffness="1" /> -->
+  </joint>
+  <joint name="fr_joint" type="fixed">
     <parent link="body_main"/>
-    <child link="right_wheel_front_steering"/>
-    <axis xyz="0 0 1"/>
-    <limit velocity="6.5" effort="1000" lower="${-pi}" upper="${pi}" />
-    <dynamics damping = "0.7"/>
-  </joint>
-  <transmission name="right_wheel_front_steering_joint_tran">
-     <type>transmission_interface/SimpleTransmission</type>
-     <joint name="right_wheel_front_steering_joint">
-       <hardwareInterface>EffortJointInterface</hardwareInterface>
-     </joint>
-     <actuator name="right_wheel_front_steering_joint_motor">
-       <hardwareInterface>EffortJointInterface</hardwareInterface>
-       <mechanicalReduction>1</mechanicalReduction>
-     </actuator>
-  </transmission>
- <link name="right_wheel_front_steering">
-    <collision>
-      <origin xyz="0 0 0" rpy="0 0 0"/>
-         <geometry>
-           <box size="0.001 0.001 0.001" />
-        </geometry>
-    </collision>
-    <visual>
-        <origin xyz="0 0 0" rpy="0 0 0"/>
-        <geometry>
-          <box size="0.001 0.001 0.001" />
-        </geometry>
-        <material name="white"/>
-    </visual>
-    <inertial>
-      <origin xyz="0 0 0" rpy="0 0 0"/>
-      <mass value="2.5"/>
-      <inertia ixx="1.0" ixy="0.0" ixz="0.0" iyy="1.0" iyz="0.0" izz="1.0" />
-    </inertial>
-  </link>
- <!-- right wheel front -->
-  <joint name="right_wheel_front_joint" type="continuous">
-    <origin xyz="0 0 0" rpy="0 0 0"/>
-    <parent link="right_wheel_front_steering"/>
-    <child link="right_wheel_front"/>
-    <axis xyz="0 1 0"/>
- <!--<limit velocity="6.5" effort="1000" lower="${-pi}" upper="${pi}" />-->
-    <dynamics damping = "0.7"/>
-  </joint>
- <!--
-  <transmission name="right_wheel_front_joint_tran">
-     <type>transmission_interface/SimpleTransmission</type>
-     <joint name="right_wheel_front_joint">
-       <hardwareInterface>EffortJointInterface</hardwareInterface>
-     </joint>
-     <actuator name="right_wheel_front_joint_motor">
-       <hardwareInterface>EffortJointInterface</hardwareInterface>
-       <mechanicalReduction>1</mechanicalReduction>
-     </actuator>
-  </transmission>
--->
- <link name="right_wheel_front">
-    <collision>
-      <origin xyz="0 0 0" rpy="0 0 0"/>
-         <geometry>
-          <mesh filename="package://erica_description/meshes/right_wheel_front.stl" scale="0.001 0.001 0.001"/>
-        </geometry>
-        <surface>
-          <friction>
-            <ode>
-              <mu>0.1</mu>
-              <mu2>1</mu2>
-            </ode>
-          </friction>
-        </surface>
-    </collision>
-    <visual>
-        <origin xyz="0 0 0" rpy="0 0 0"/>
-        <geometry>
-          <mesh filename="package://erica_description/meshes/right_wheel_front.stl" scale="0.001 0.001 0.001"/>
-        </geometry>
-        <material name="white"/>
-    </visual>
-    <inertial>
-      <origin xyz="0 0 0" rpy="0 0 0"/>
-      <mass value="1"/>
-      <inertia ixx="1.0" ixy="0.0" ixz="0.0" iyy="1.0" iyz="0.0" izz="1.0" />
-    </inertial>
-  </link>
-  <!-- left wheel rear steering-->
-  <joint name="left_wheel_rear_steering_joint" type="revolute">
-    <origin xyz="-0.09 0.157 0.037" rpy="0 0 0"/>
+    <child link="fr_link"/>
+    <origin rpy="0 0 0" xyz="${base_length/2 - wheel_setback} ${-base_width/2 - wheel_gap} 0.0"/>
+    <axis xyz="0 0 0"/>
+    <!-- <dynamics damping="1.0" friction="0.0" spring_stiffness="1" /> -->
+  </joint>
+  <joint name="bl_joint" type="fixed">
     <parent link="body_main"/>
-    <child link="left_wheel_rear_steering"/>
-    <axis xyz="0 0 1"/>
-    <limit velocity="6.5" effort="1000" lower="${-pi}" upper="${pi}" />
-    <dynamics damping = "0.7"/>
-  </joint>
-  <transmission name="left_wheel_rear_steering_joint_tran">
-     <type>transmission_interface/SimpleTransmission</type>
-     <joint name="left_wheel_rear_steering_joint">
-       <hardwareInterface>EffortJointInterface</hardwareInterface>
-     </joint>
-     <actuator name="left_wheel_rear_steering_joint_motor">
-       <hardwareInterface>EffortJointInterface</hardwareInterface>
-       <mechanicalReduction>1</mechanicalReduction>
-     </actuator>
-  </transmission>
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
Commit message: modified

File: erica_description/urdf/erica_robot.xacro (robot description, xacro)
@@ -30,5 +30,5 @@
     <inertial>
       <origin xyz="0 0 0" rpy="0 0 0"/>
-      <mass value="50"/>
+      <mass value="10"/>
       <inertia ixx="1.0" ixy="0.0" ixz="0.0" iyy="1.0" iyz="0.0" izz="1.0" />
     </inertial>
@@ -74,5 +74,5 @@
     </collision>
     <inertial>
-      <mass value="2" />
+      <mass value="20" />
       <origin rpy="${pi/2} 0 0" xyz="0 0 0"/>
       <inertia ixx="1e-6" ixy="0" ixz="0" iyy="1e-6" iyz="0" izz="1e-6" />
@@ -93,5 +93,5 @@
     </collision>
     <inertial>
-      <mass value="2" />
+      <mass value="20" />
       <origin rpy="${pi/2} 0 0" xyz="0 0 0"/>
       <inertia ixx="1e-6" ixy="0" ixz="0" iyy="1e-6" iyz="0" izz="1e-6" />
@@ -112,5 +112,5 @@
     </collision>
     <inertial>
-      <mass value="2" />
+      <mass value="20" />
       <origin rpy="${pi/2} 0 0" xyz="0 0 0"/>
       <inertia ixx="1e-6" ixy="0" ixz="0" iyy="1e-6" iyz="0" izz="1e-6" />
@@ -131,5 +131,5 @@
     </collision>
     <inertial>
-      <mass value="2" />
+      <mass value="20" />
       <origin rpy="${pi/2} 0 0" xyz="0 0 0"/>
       <inertia ixx="1e-6" ixy="0" ixz="0" iyy="1e-6" iyz="0" izz="1e-6" />
@@ -186,5 +186,5 @@
     <inertial>
       <origin xyz="0 0 0" rpy="0 0 0"/>
-      <mass value="1"/>
+      <mass value="0.1"/>
       <inertia ixx="1.0" ixy="0.0" ixz="0.0" iyy="1.0" iyz="0.0" izz="1.0" />
     </inertial>
@@ -225,5 +225,5 @@
     <inertial>
       <origin xyz="0 0 0" rpy="0 0 0"/>
-      <mass value="1"/>
+      <mass value="0.1"/>
       <inertia ixx="1.0" ixy="0.0" ixz="0.0" iyy="1.0" iyz="0.0" izz="1.0" />
     </inertial>
@@ -264,5 +264,5 @@
     <inertial>
       <origin xyz="0 0 0" rpy="0 0 0"/>
-      <mass value="1"/>
+      <mass value="0.1"/>
       <inertia ixx="1.0" ixy="0.0" ixz="0.0" iyy="1.0" iyz="0.0" izz="1.0" />
     </inertial>
@@ -303,5 +303,5 @@
     <inertial>
       <origin xyz="0 0 0" rpy="0 0 0"/>
-      <mass value="1"/>
+      <mass value="0.1"/>
       <inertia ixx="1.0" ixy="0.0" ixz="0.0" iyy="1.0" iyz="0.0" izz="1.0" />
     </inertial>
@@ -330,5 +330,5 @@
     <inertial>
       <origin xyz="0 0 0" rpy="0 0 0"/>
-      <mass value="1"/>
+      <mass value="0.1"/>
       <inertia ixx="1.0" ixy="0.0" ixz="0.0" iyy="1.0" iyz="0.0" izz="1.0" />
     </inertial>
@@ -396,5 +396,5 @@
     <inertial>
       <origin xyz="0 0 0" rpy="0 0 0"/>
-      <mass value="1"/>
+      <mass value="0.1"/>
       <inertia ixx="1.0" ixy="0.0" ixz="0.0" iyy="1.0" iyz="0.0" izz="1.0" />
     </inertial>
@@ -435,5 +435,5 @@
     <inertial>
       <origin xyz="0 0 0" rpy="0 0 0"/>
-      <mass value="1"/>
+      <mass value="0.1"/>
       <inertia ixx="1.0" ixy="0.0" ixz="0.0" iyy="1.0" iyz="0.0" izz="1.0" />
     </inertial>
@@ -474,5 +474,5 @@
     <inertial>
       <origin xyz="0 0 0" rpy="0 0 0"/>
-      <mass value="1"/>
+      <mass value="0.1"/>
       <inertia ixx="1.0" ixy="0.0" ixz="0.0" iyy="1.0" iyz="0.0" izz="1.0" />
     </inertial>
@@ -513,5 +513,5 @@
     <inertial>
       <origin xyz="0 0 0" rpy="0 0 0"/>
-      <mass value="1"/>
+      <mass value="0.1"/>
       <inertia ixx="1.0" ixy="0.0" ixz="0.0" iyy="1.0" iyz="0.0" izz="1.0" />
     </inertial>
@@ -552,5 +552,5 @@
     <inertial>
       <origin xyz="0 0 0" rpy="0 0 0"/>
-      <mass value="1"/>
+      <mass value="0.1"/>
       <inertia ixx="1.0" ixy="0.0" ixz="0.0" iyy="1.0" iyz="0.0" izz="1.0" />
     </inertial>
@@ -591,5 +591,5 @@
     <inertial>
       <origin xyz="0 0 0" rpy="0 0 0"/>
-      <mass value="1"/>
+      <mass value="0.1"/>
       <inertia ixx="1.0" ixy="0.0" ixz="0.0" iyy="1.0" iyz="0.0" izz="1.0" />
     </inertial>
@@ -631,5 +631,5 @@
     <inertial>
       <origin xyz="0 0 0" rpy="0 0 0"/>
-      <mass value="1"/>
+      <mass value="0.1"/>
       <inertia ixx="1.0" ixy="0.0" ixz="0.0" iyy="1.0" iyz="0.0" izz="1.0" />
     </inertial>
@@ -670,5 +670,5 @@
     <inertial>
       <origin xyz="0 0 0" rpy="0 0 0"/>
-      <mass value="1"/>
+      <mass value="0.1"/>
       <inertia ixx="1.0" ixy="0.0" ixz="0.0" iyy="1.0" iyz="0.0" izz="1.0" />
     </inertial>
@@ -709,5 +709,5 @@
     <inertial>
       <origin xyz="0 0 0" rpy="0 0 0"/>
-      <mass value="1"/>
+      <mass value="0.1"/>
       <inertia ixx="1.0" ixy="0.0" ixz="0.0" iyy="1.0" iyz="0.0" izz="1.0" />
     </inertial>
@@ -748,5 +748,5 @@
     <inertial>
       <origin xyz="0 0 0" rpy="0 0 0"/>
-      <mass value="1"/>
+      <mass value="0.1"/>
       <inertia ixx="1.0" ixy="0.0" ixz="0.0" iyy="1.0" iyz="0.0" izz="1.0" />
     </inertial>
@@ -787,5 +787,5 @@
     <inertial>
       <origin xyz="0 0 0" rpy="0 0 0"/>
-      <mass value="1"/>
+      <mass value="0.1"/>
       <inertia ixx="1.0" ixy="0.0" ixz="0.0" iyy="1.0" iyz="0.0" izz="1.0" />
     </inertial>
@@ -826,5 +826,5 @@
     <inertial>
       <origin xyz="0 0 0" rpy="0 0 0"/>
-      <mass value="1"/>
+      <mass value="0.1"/>
       <inertia ixx="1.0" ixy="0.0" ixz="0.0" iyy="1.0" iyz="0.0" izz="1.0" />
     </inertial>
